File: cpu/tinycom-cpu.kicad_pcb (KiCad board)
At the start: 4 copper layers, 39.4 x 41.4 mm, 23 parts, among them P1 CONN_02X08, P2 CONN_02X08, U1 IC_A13, U2 H5TQ2G83BFR/FBGA82, Y1 Crystal

Commit message: adjust
Routing:
- net VCC_33: track 31.6 -> 30.6 mm
- net UART1_TX: track 37.4 -> 36.8 mm
Changed lines of the file:
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@@
     (thickness 1.6)
     (drawings 23)
-    (tracks 1049)
+    (tracks 1045)
     (zones 0)
     (modules 23)
@@
   (segment (start 114.3 137.588256) (end 114.379744 137.668) (width 0.15) (layer F.Cu) (net 92))
   (via (at 114.379744 137.668) (size 0.6) (drill 0.3) (layers F.Cu B.Cu) (net 92))
-  (segment (start 102.108 154.432) (end 112.138999 144.401001) (width 0.15) (layer B.Cu) (net 93))
   (segment (start 96.266 156.464) (end 98.298 154.432) (width 0.15) (layer B.Cu) (net 93))
   (segment (start 98.298 154.432) (end 102.108 154.432) (width 0.15) (layer B.Cu) (net 93))
-  (segment (start 112.138999 144.246999) (end 112.740552 144.848552) (width 0.15) (layer B.Cu) (net 93))
-  (segment (start 112.138999 144.401001) (end 112.138999 144.246999) (width 0.15) (layer B.Cu) (net 93))
-  (segment (start 112.740552 144.848552) (end 112.92696 144.848552) (width 0.15) (layer B.Cu) (net 93))
+  (segment (start 102.108 154.432) (end 111.691447 144.848553) (width 0.15) (layer B.Cu) (net 93))
+  (segment (start 111.691447 144.848553) (end 112.92696 144.848552) (width 0.15) (layer B.Cu) (net 93))
   (segment (start 112.92696 144.848552) (end 113.267271 144.508241) (width 0.15) (layer B.Cu) (net 93))
   (segment (start 113.411 137.795) (end 114.757831 139.141831) (width 0.15) (layer B.Cu) (net 93))
@@
   (segment (start 106.683842 150.117842) (end 105.664 149.098) (width 0.15) (layer F.Cu) (net 99))
   (via (at 105.664 149.098) (size 0.6) (drill 0.3) (layers F.Cu B.Cu) (net 99))
+  (segment (start 106.436221 151.868812) (end 106.719997 152.152588) (width 0.15) (layer F.Cu) (net 100))
   (segment (start 103.886 159.004) (end 102.722399 157.840399) (width 0.3) (layer F.Cu) (net 100))
   (segment (start 102.722399 157.840399) (end 102.722399 154.434601) (width 0.3) (layer F.Cu) (net 100))
@@
   (segment (start 105.340864 152.330864) (end 105.358385 152.348385) (width 0.15) (layer F.Cu) (net 100))
   (segment (start 105.870465 151.303056) (end 105.340864 151.832657) (width 0.15) (layer F.Cu) (net 100))
-  (segment (start 105.782649 152.348385) (end 105.358385 152.348385) (width 0.15) (layer F.Cu) (net 100))
   (segment (start 105.90662 152.398413) (end 105.408413 152.398413) (width 0.15) (layer F.Cu) (net 100))
-  (segment (start 106.479905 152.152588) (end 106.284108 152.348385) (width 0.15) (layer F.Cu) (net 100))
-  (segment (start 106.719997 152.152588) (end 106.479905 152.152588) (width 0.15) (layer F.Cu) (net 100))
   (via (at 105.358385 152.348385) (size 0.6) (drill 0.3) (layers F.Cu B.Cu) (net 100))
-  (segment (start 106.284108 152.348385) (end 105.782649 152.348385) (width 0.15) (layer F.Cu) (net 100))
   (segment (start 105.340864 151.832657) (end 105.340864 152.330864) (width 0.15) (layer F.Cu) (net 100))
   (segment (start 106.436221 151.868812) (end 105.90662 152.398413) (width 0.15) (layer F.Cu) (net 100))
@@
   (segment (start 96.541871 136.528834) (end 96.576134 136.563097) (width 0.15) (layer F.Cu) (net 122))
   (segment (start 96.576134 136.563097) (end 97.105735 137.092698) (width 0.15) (layer F.Cu) (net 122))
+  (segment (start 95.061404 137.476755) (end 95.649886 136.888273) (width 0.15) (layer F.Cu) (net 123))
+  (segment (start 96.292358 136.846873) (end 96.821959 137.376474) (width 0.15) (layer F.Cu) (net 123))
+  (segment (start 95.649886 136.888273) (end 95.649886 136.887114) (width 0.15) (layer F.Cu) (net 123))
+  (segment (start 95.649886 136.887114) (end 95.708156 136.828844) (width 0.15) (layer F.Cu) (net 123))
+  (segment (start 95.708156 136.828844) (end 96.274329 136.828844) (width 0.15) (layer F.Cu) (net 123))
+  (segment (start 96.274329 136.828844) (end 96.292358 136.846873) (width 0.15) (layer F.Cu) (net 123))
   (segment (start 94.920265 137.617894) (end 95.061404 137.476755) (width 0.15) (layer F.Cu) (net 123))
   (segment (start 94.39351 137.76249) (end 94.775669 137.76249) (width 0.15) (layer F.Cu) (net 123))
-  (segment (start 95.061404 137.476755) (end 95.649886 136.888273) (width 0.15) (layer F.Cu) (net 123))
   (segment (start 93.477323 137.762499) (end 94.393501 137.762499) (width 0.15) (layer F.Cu) (net 123))
   (segment (start 94.393501 137.762499) (end 94.39351 137.76249) (width 0.15) (layer F.Cu) (net 123))
   (segment (start 94.775669 137.76249) (end 95.061404 137.476755) (width 0.15) (layer F.Cu) (net 123))
-  (segment (start 96.292358 136.846873) (end 96.821959 137.376474) (width 0.15) (layer F.Cu) (net 123))
-  (segment (start 95.835156 136.828844) (end 96.274329 136.828844) (width 0.15) (layer F.Cu) (net 123))
-  (segment (start 95.775727 136.888273) (end 95.835156 136.828844) (width 0.15) (layer F.Cu) (net 123))
   (segment (start 92.8846 138.16) (end 93.079822 138.16) (width 0.15) (layer F.Cu) (net 123))
   (segment (start 93.079822 138.16) (end 93.477323 137.762499) (width 0.15) (layer F.Cu) (net 123))
-  (segment (start 95.649886 136.888273) (end 95.775727 136.888273) (width 0.15) (layer F.Cu) (net 123))
-  (segment (start 96.274329 136.828844) (end 96.292358 136.846873) (width 0.15) (layer F.Cu) (net 123))
   (segment (start 94.787594 138.812521) (end 95.220276 138.379839) (width 0.15) (layer F.Cu) (net 124))
   (segment (start 95.220276 137.742162) (end 95.774154 137.188284) (width 0.15) (layer F.Cu) (net 124))
@@
   (segment (start 92.482001 142.558001) (end 92.246015 142.322015) (width 0.15) (layer F.Cu) (net 126))
   (segment (start 92.246015 142.322015) (end 92.0845 142.1605) (width 0.15) (layer F.Cu) (net 126))
-  (segment (start 96.16208 143.906259) (end 96.301762 143.906259) (width 0.15) (layer F.Cu) (net 127))
-  (segment (start 96.301762 143.906259) (end 97.387715 142.820306) (width 0.15) (layer F.Cu) (net 127))
+  (segment (start 96.301762 143.906259) (end 96.356457 143.851564) (width 0.15) (layer F.Cu) (net 127))
+  (segment (start 96.16208 144.385023) (end 96.16208 144.045941) (width 0.15) (layer F.Cu) (net 127))
+  (segment (start 96.356457 143.851564) (end 97.387715 142.820306) (width 0.15) (layer F.Cu) (net 127))
+  (segment (start 96.16208 144.045941) (end 96.356457 143.851564) (width 0.15) (layer F.Cu) (net 127))
   (segment (start 95.88908 144.658023) (end 96.16208 144.385023) (width 0.15) (layer F.Cu) (net 127))
-  (segment (start 96.16208 144.385023) (end 96.16208 143.906259) (width 0.15) (layer F.Cu) (net 127))
   (segment (start 94.861514 144.26079) (end 95.258747 144.658023) (width 0.15) (layer F.Cu) (net 127))
   (segment (start 95.258747 144.658023) (end 95.88908 144.658023) (width 0.15) (layer F.Cu) (net 127))
@@
   (segment (start 93.875501 144.163299) (end 93.972992 144.26079) (width 0.15) (layer F.Cu) (net 127))
   (segment (start 93.972992 144.26079) (end 94.861514 144.26079) (width 0.15) (layer F.Cu) (net 127))
+  (segment (start 96.52 144.451381) (end 96.52 144.255573) (width 0.15) (layer F.Cu) (net 128))
+  (segment (start 96.52 144.255573) (end 96.663274 144.112299) (width 0.15) (layer F.Cu) (net 128))
   (segment (start 94.675056 144.958301) (end 94.675056 144.968564) (width 0.15) (layer F.Cu) (net 128))
   (segment (start 94.675056 144.968564) (end 95.414526 145.708034) (width 0.15) (layer F.Cu) (net 128))
@@
   (segment (start 96.29987 145.435034) (end 96.29987 144.671511) (width 0.15) (layer F.Cu) (net 128))
   (segment (start 96.29987 144.671511) (end 96.52 144.451381) (width 0.15) (layer F.Cu) (net 128))
-  (segment (start 96.52 144.451381) (end 96.52 144.112299) (width 0.15) (layer F.Cu) (net 128))
-  (segment (start 96.52 144.112299) (end 96.663274 144.112299) (width 0.15) (layer F.Cu) (net 128))
   (segment (start 96.663274 144.112299) (end 97.671491 143.104082) (width 0.15) (layer F.Cu) (net 128))
   (segment (start 94.675056 144.958301) (end 94.675056 144.960165) (width 0.15) (layer F.Cu) (net 128))
