File: cpu/tinycom-cpu.sch (KiCad schematic (older format))
At the start: 23 parts, among them P1 CONN_02X08, P2 CONN_02X08, U1 OLIMEX_IC_A13, U2 H5TQ2G83BFR/FBGA82, Y1 Crystal

Commit message: xxx
Connections:
- net GND: now also U1.79 (AGND), U1.GND_ (GND)
Changed lines of the file:
@@
 $EndComp
 $Comp
-L GND #PWR02
+L GND #PWR01
 U 1 1 5624C74D
 P 6400 5750
-F 0 "#PWR02" H 6400 5500 50  0001 C CNN
+F 0 "#PWR01" H 6400 5500 50  0001 C CNN
 F 1 "GND" H 6400 5600 50  0000 C CNN
 F 2 "" H 6400 5750 60  0000 C CNN
@@
 $EndComp
 $Comp
-L GND #PWR03
+L GND #PWR02
 U 1 1 5624C778
 P 6400 6050
-F 0 "#PWR03" H 6400 5800 50  0001 C CNN
+F 0 "#PWR02" H 6400 5800 50  0001 C CNN
 F 1 "GND" H 6400 5900 50  0000 C CNN
 F 2 "" H 6400 6050 60  0000 C CNN
@@
 VCC_14
 $Comp
-L +3.3V #PWR04
+L +3.3V #PWR03
 U 1 1 5624CB40
 P 7400 2200
-F 0 "#PWR04" H 7400 2050 50  0001 C CNN
+F 0 "#PWR03" H 7400 2050 50  0001 C CNN
 F 1 "+3.3V" H 7400 2340 50  0000 C CNN
 F 2 "" H 7400 2200 60  0000 C CNN
@@
 $EndComp
 $Comp
-L +1V5 #PWR05
+L +1V5 #PWR04
 U 1 1 5624CB62
 P 5250 2150
-F 0 "#PWR05" H 5250 2000 50  0001 C CNN
+F 0 "#PWR04" H 5250 2000 50  0001 C CNN
 F 1 "+1V5" H 5250 2290 50  0000 C CNN
 F 2 "" H 5250 2150 60  0000 C CNN
@@
 DDR3_BA2
 $Comp
-L +1V5 #PWR06
+L +1V5 #PWR05
 U 1 1 5625F72C
 P 15200 3600
-F 0 "#PWR06" H 15200 3450 50  0001 C CNN
+F 0 "#PWR05" H 15200 3450 50  0001 C CNN
 F 1 "+1V5" H 15200 3740 50  0000 C CNN
 F 2 "" H 15200 3600 60  0000 C CNN
@@
 $EndComp
 $Comp
-L GND #PWR07
+L GND #PWR06
 U 1 1 5625F96A
 P 15350 7200
-F 0 "#PWR07" H 15350 6950 50  0001 C CNN
+F 0 "#PWR06" H 15350 6950 50  0001 C CNN
 F 1 "GND" H 15350 7050 50  0000 C CNN
 F 2 "" H 15350 7200 60  0000 C CNN
@@
 DDR3_RST
 $Comp
-L GND #PWR08
+L GND #PWR07
 U 1 1 5625FBB8
 P 11800 5950
-F 0 "#PWR08" H 11800 5700 50  0001 C CNN
+F 0 "#PWR07" H 11800 5700 50  0001 C CNN
 F 1 "GND" H 11800 5800 50  0000 C CNN
 F 2 "" H 11800 5950 60  0000 C CNN
@@
 $EndComp
 $Comp
-L +1V5 #PWR09
+L +1V5 #PWR08
 U 1 1 5625FE07
 P 12000 7100
-F 0 "#PWR09" H 12000 6950 50  0001 C CNN
+F 0 "#PWR08" H 12000 6950 50  0001 C CNN
 F 1 "+1V5" H 12000 7240 50  0000 C CNN
 F 2 "" H 12000 7100 60  0000 C CNN
@@
 $EndComp
 $Comp
-L GND #PWR010
+L GND #PWR09
 U 1 1 5625FF1B
 P 12000 7850
-F 0 "#PWR010" H 12000 7600 50  0001 C CNN
+F 0 "#PWR09" H 12000 7600 50  0001 C CNN
 F 1 "GND" H 12000 7700 50  0000 C CNN
 F 2 "" H 12000 7850 60  0000 C CNN
@@
 $EndComp
 $Comp
-L GND #PWR011
+L GND #PWR010
 U 1 1 56260662
 P 12250 8100
-F 0 "#PWR011" H 12250 7850 50  0001 C CNN
+F 0 "#PWR010" H 12250 7850 50  0001 C CNN
 F 1 "GND" H 12250 7950 50  0000 C CNN
 F 2 "" H 12250 8100 60  0000 C CNN
@@
 NoConn ~ 15100 7350
 $Comp
-L GND #PWR012
+L GND #PWR011
 U 1 1 56261679
 P 12450 7900
-F 0 "#PWR012" H 12450 7650 50  0001 C CNN
+F 0 "#PWR011" H 12450 7650 50  0001 C CNN
 F 1 "GND" H 12450 7750 50  0000 C CNN
 F 2 "" H 12450 7900 60  0000 C CNN
@@
 $EndComp
 $Comp
-L GND #PWR015
+L GND #PWR012
 U 1 1 56262D84
 P 11100 7950
-F 0 "#PWR015" H 11100 7700 50  0001 C CNN
+F 0 "#PWR012" H 11100 7700 50  0001 C CNN
 F 1 "GND" H 11100 7800 50  0000 C CNN
 F 2 "" H 11100 7950 60  0000 C CNN
@@
 $EndComp
 $Comp
-L +1V5 #PWR016
+L +1V5 #PWR013
 U 1 1 562642D9
 P 16050 3500
-F 0 "#PWR016" H 16050 3350 50  0001 C CNN
+F 0 "#PWR013" H 16050 3350 50  0001 C CNN
 F 1 "+1V5" H 16050 3640 50  0000 C CNN
 F 2 "" H 16050 3500 60  0000 C CNN
@@
 $EndComp
 $Comp
-L GND #PWR017
+L GND #PWR014
 U 1 1 562643A7
 P 16100 3900
-F 0 "#PWR017" H 16100 3650 50  0001 C CNN
+F 0 "#PWR014" H 16100 3650 50  0001 C CNN
 F 1 "GND" H 16100 3750 50  0000 C CNN
 F 2 "" H 16100 3900 60  0000 C CNN
@@
 $EndComp
 $Comp
-L GND #PWR018
+L GND #PWR015
 U 1 1 56265943
 P 6850 3500
-F 0 "#PWR018" H 6850 3250 50  0001 C CNN
+F 0 "#PWR015" H 6850 3250 50  0001 C CNN
 F 1 "GND" H 6850 3350 50  0000 C CNN
 F 2 "" H 6850 3500 60  0000 C CNN
@@
 $EndComp
 $Comp
-L GND #PWR019
+L GND #PWR016
 U 1 1 56265988
 P 7050 2700
-F 0 "#PWR019" H 7050 2450 50  0001 C CNN
+F 0 "#PWR016" H 7050 2450 50  0001 C CNN
 F 1 "GND" H 7050 2550 50  0000 C CNN
 F 2 "" H 7050 2700 60  0000 C CNN
@@
 Text GLabel 12000 7500 0    60   Input ~ 0
 SVREF
+$Comp
+L GND #PWR?
+U 1 1 562A3A06
+P 7100 5400
+F 0 "#PWR?" H 7100 5150 50  0001 C CNN
+F 1 "GND" H 7100 5250 50  0000 C CNN
+F 2 "" H 7100 5400 60  0000 C CNN
+F 3 "" H 7100 5400 60  0000 C CNN
+	1    7100 5400
+	1    0    0    -1
+$EndComp
+Wire Wire Line
+	7100 5400 7300 5400
+Connection ~ 7300 5400
 $EndSCHEMATC
