File: cpu/tinycom-cpu.sch (KiCad schematic (older format))
At the start: 23 parts, among them P1 CONN_02X08, P2 CONN_02X08, U1 OLIMEX_IC_A13, U2 H5TQ2G83BFR/FBGA82, Y1 Crystal

Commit message: fix
Connections:
- net +3V3: no longer U1.80 (VRP), U1.82 (VRA2), U1.83 (VRA1)
Changed lines of the file:
@@
 Text GLabel 4550 2200 0    60   Input ~ 0
 VCC_30
-Text GLabel 7300 6550 0    60   Input ~ 0
+Text GLabel 7500 7150 0    60   Input ~ 0
 VCC_33
 Text GLabel 7500 8350 0    60   Input ~ 0
@@
 	7300 5350 7500 5350
 Wire Wire Line
-	7500 6550 7300 6550
-Wire Wire Line
-	7300 6550 7300 7150
-Wire Wire Line
-	7300 7150 7500 7150
-Wire Wire Line
-	7500 6850 7300 6850
-Connection ~ 7300 6850
-Wire Wire Line
-	7500 6750 7300 6750
-Connection ~ 7300 6750
-Wire Wire Line
 	7500 5750 7350 5750
