File: tinycom-a20/_saved_tinycom-a20.sch (KiCad schematic (older format))
At the start: 7 parts, among them P1 CONN_02X08, U1 ALLWINNERA10/TFBGA441, U2 H5TQG63BFR/FBGA96

Commit message: ddr3 routing
Parts:
- gave numbers to parts that had none: 1
Changed lines of the file:
@@
 $EndComp
 $Comp
-L CONN_02X08 P?
+L CONN_02X08 P2
 U 1 1 563EFECC
 P 20600 9800
-F 0 "P?" H 20600 10250 50  0000 C CNN
+F 0 "P2" H 20600 10250 50  0000 C CNN
 F 1 "CONN_02X08" V 20600 9800 50  0000 C CNN
 F 2 "Socket_Strips:Socket_Strip_Straight_2x08" H 20600 8600 60  0001 C CNN
