File: tinycom-a20/tinycom-a20.sch (KiCad schematic (older format))
At the start: 7 parts, among them P1 CONN_02X08, U1 ALLWINNERA10/TFBGA441, U2 H5TQG63BFR/FBGA96

Commit message: before change track width
Parts:
- added U3: H27UBG8T2A/TSOP48, tsop48:TSOP48, symbol H27UBG8T2A/TSOP48
- gave numbers to parts that had none: 1
Connections:
- net ND7: now reaches U1.G20 (ND7/SDC1_D3/PC15)
- net ND7: now also U3.44 (I/O7)
- net ND6: now reaches U1.G21 (ND6/SDC1_D2/PC14)
- net ND6: now also U3.43 (I/O6)
- net ND3: now reaches U1.G22 (ND3/SDC2_D3/PC11)
- net ND3: now also U3.32 (I/O3)
- net ND2: now reaches U1.G23 (ND2/SDC2_D2/PC10)
- net ND2: now also U3.31 (I/O2)
- net ND5: now reaches U1.H20 (ND5/SDC1_D1/PC13)
- net ND5: now also U3.42 (I/O5)
- net ND4: now reaches U1.H21 (ND4/SDC1_D0/PC12)
- net ND4: now also U3.41 (I/O4)
- net ND1: now reaches U1.H22 (ND1/SDC2_D1/PC9)
- net ND1: now also U3.30 (I/O1)
- net ND0: now reaches U1.H23 (ND0/SDC2_D0/PC8)
- net ND0: now also U3.29 (I/O0)
- net NRB0: now reaches U1.J23 (NRB0/SDC2_CMD/PC6)
- net NRB0: now also U3.7 (R/B#)
- net NRE#: now reaches U1.K22 (NRE#/PC5)
- net NRE#: now also U3.8 (RE#)
- net NCLE: now reaches U1.L23 (NCLE/SPI0_CLK/PC2)
- net NCLE: now also U3.16 (CLE)
- net NALE: now reaches U1.M22 (NALE/SPI0_MISO/PC1)
- net NALE: now also U3.17 (ALE)
- net NWE#: now reaches U1.M23 (NWE#/SPIO_MOSI/PC0)
- net NWE#: now also U3.18 (WE#)
Changed lines of the file:
@@
 $EndComp
 $Comp
-L GND #PWR8
+L GND #PWR01
 U 1 1 563E445F
 P 21050 6550
-F 0 "#PWR8" H 21050 6300 50  0001 C CNN
+F 0 "#PWR01" H 21050 6300 50  0001 C CNN
 F 1 "GND" H 21050 6400 50  0000 C CNN
 F 2 "" H 21050 6550 60  0000 C CNN
@@
 SCK_P
 $Comp
-L GND #PWR5
+L GND #PWR02
 U 1 1 563ECE56
 P 18200 1250
-F 0 "#PWR5" H 18200 1000 50  0001 C CNN
+F 0 "#PWR02" H 18200 1000 50  0001 C CNN
 F 1 "GND" H 18200 1100 50  0000 C CNN
 F 2 "" H 18200 1250 60  0000 C CNN
@@
 $EndComp
 $Comp
-L +1V5 #PWR6
+L +1V5 #PWR03
 U 1 1 563ED4AE
 P 19800 1100
-F 0 "#PWR6" H 19800 950 50  0001 C CNN
+F 0 "#PWR03" H 19800 950 50  0001 C CNN
 F 1 "+1V5" H 19800 1240 50  0000 C CNN
 F 2 "" H 19800 1100 60  0000 C CNN
@@
 $EndComp
 $Comp
-L +1V5 #PWR7
+L +1V5 #PWR04
 U 1 1 563ED57F
 P 19800 7250
-F 0 "#PWR7" H 19800 7100 50  0001 C CNN
+F 0 "#PWR04" H 19800 7100 50  0001 C CNN
 F 1 "+1V5" H 19800 7390 50  0000 C CNN
 F 2 "" H 19800 7250 60  0000 C CNN
@@
 $EndComp
 $Comp
-L +1V5 #PWR1
+L +1V5 #PWR05
 U 1 1 563EDD3D
 P 16850 5600
-F 0 "#PWR1" H 16850 5450 50  0001 C CNN
+F 0 "#PWR05" H 16850 5450 50  0001 C CNN
 F 1 "+1V5" H 16850 5740 50  0000 C CNN
 F 2 "" H 16850 5600 60  0000 C CNN
@@
 $EndComp
 $Comp
-L GND #PWR2
+L GND #PWR06
 U 1 1 563EDF36
 P 16850 6300
-F 0 "#PWR2" H 16850 6050 50  0001 C CNN
+F 0 "#PWR06" H 16850 6050 50  0001 C CNN
 F 1 "GND" H 16850 6150 50  0000 C CNN
 F 2 "" H 16850 6300 60  0000 C CNN
@@
 $EndComp
 $Comp
-L GND #PWR3
+L GND #PWR07
 U 1 1 563EE398
 P 17600 5550
-F 0 "#PWR3" H 17600 5300 50  0001 C CNN
+F 0 "#PWR07" H 17600 5300 50  0001 C CNN
 F 1 "GND" H 17600 5400 50  0000 C CNN
 F 2 "" H 17600 5550 60  0000 C CNN
@@
 Connection ~ 17650 2250
 $Comp
-L +1V5 #PWR4
+L +1V5 #PWR08
 U 1 1 563EF32F
 P 17650 2100
-F 0 "#PWR4" H 17650 1950 50  0001 C CNN
+F 0 "#PWR08" H 17650 1950 50  0001 C CNN
 F 1 "+1V5" H 17650 2240 50  0000 C CNN
 F 2 "" H 17650 2100 60  0000 C CNN
@@
 $EndComp
 $Comp
-L CONN_02X08 P?
+L CONN_02X08 P2
 U 1 1 563EFECC
 P 20600 9800
-F 0 "P?" H 20600 10250 50  0000 C CNN
+F 0 "P2" H 20600 10250 50  0000 C CNN
 F 1 "CONN_02X08" V 20600 9800 50  0000 C CNN
 F 2 "Socket_Strips:Socket_Strip_Straight_2x08" H 20600 8600 60  0001 C CNN
@@
 	1    0    0    -1
 $EndComp
+$Comp
+L H27UBG8T2A/TSOP48 U3
+U 1 1 563F0202
+P 20100 12250
+F 0 "U3" H 19700 13675 50  0000 L BNN
+F 1 "H27UBG8T2A/TSOP48" H 19700 10750 50  0000 L BNN
+F 2 "tsop48:TSOP48" H 20100 12400 50  0001 C CNN
+F 3 "" H 20100 12250 60  0000 C CNN
+	1    20100 12250
+	1    0    0    -1
+$EndComp
+Text GLabel 11650 9950 2    60   Input ~ 0
+ND0
+Text GLabel 11650 10050 2    60   Input ~ 0
+ND1
+Text GLabel 11650 10150 2    60   Input ~ 0
+ND2
+Text GLabel 11650 10250 2    60   Input ~ 0
+ND3
+Text GLabel 11650 10350 2    60   Input ~ 0
+ND4
+Text GLabel 11650 10450 2    60   Input ~ 0
+ND5
+Text GLabel 11650 10550 2    60   Input ~ 0
+ND6
+Text GLabel 11650 10650 2    60   Input ~ 0
+ND7
+Text GLabel 11650 9750 2    60   Input ~ 0
+NRB0
+Text GLabel 11650 9150 2    60   Input ~ 0
+NWE#
+Text GLabel 11650 9650 2    60   Input ~ 0
+NRE#
+Text GLabel 11650 9250 2    60   Input ~ 0
+NALE
+Text GLabel 11650 9350 2    60   Input ~ 0
+NCLE
+Text GLabel 20700 12250 2    60   Input ~ 0
+ND0
+Text GLabel 20700 12350 2    60   Input ~ 0
+ND1
+Text GLabel 20700 12450 2    60   Input ~ 0
+ND2
+Text GLabel 20700 12550 2    60   Input ~ 0
+ND3
+Text GLabel 20700 12650 2    60   Input ~ 0
+ND4
+Text GLabel 20700 12750 2    60   Input ~ 0
+ND5
+Text GLabel 20700 12850 2    60   Input ~ 0
+ND6
+Text GLabel 20700 12950 2    60   Input ~ 0
+ND7
+Text GLabel 19500 13450 0    60   Input ~ 0
+NALE
+Text GLabel 19500 13550 0    60   Input ~ 0
+NCLE
+Text GLabel 19500 13150 0    60   Input ~ 0
+NWE#
+Text GLabel 19500 12950 0    60   Input ~ 0
+NRB0
+Text GLabel 19500 12850 0    60   Input ~ 0
+NRE#
 $EndSCHEMATC

Commit message: hardware license
Parts:
- added C1, C2: C_Small, Capacitors_SMD:C_0603_HandSoldering, symbol C_Small
- added Y1: Crystal_Small, opendous:Crystal_5x3.2mm, symbol Crystal_Small
- R1, R2, R3: footprint Resistors_SMD:R_0603 -> Resistors_SMD:R_0603_HandSoldering
Connections:
- net GND: now also C1.2, C2.2
- net at U1.N22 (CLK24M_OUT): now also C2.1, Y1.1
- net at U1.N23 (CLK24M_IN): now also C1.1, Y1.2
Other:
- moved on the sheet: U1E
Changed lines of the file:
@@
 F 0 "R1" H 20730 6470 50  0000 L CNN
 F 1 "R_Small" H 20730 6410 50  0000 L CNN
-F 2 "Resistors_SMD:R_0603" H 20700 6450 60  0001 C CNN
+F 2 "Resistors_SMD:R_0603_HandSoldering" H 20700 6450 60  0001 C CNN
 F 3 "" H 20700 6450 60  0000 C CNN
 	1    20700 6450
@@
 L ALLWINNERA10/TFBGA441 U1
 U 5 1 563E5534
-P 14900 11800
-F 0 "U1" H 14900 11800 60  0000 C CNN
-F 1 "ALLWINNERA10/TFBGA441" H 14900 11650 60  0000 C CNN
-F 2 "441fbga-p08:441TFBGA-P0.8" H 14900 11800 60  0001 C CNN
-F 3 "" H 14900 11800 60  0000 C CNN
-	5    14900 11800
+P 15300 11750
+F 0 "U1" H 15300 11750 60  0000 C CNN
+F 1 "ALLWINNERA10/TFBGA441" H 15300 11600 60  0000 C CNN
+F 2 "441fbga-p08:441TFBGA-P0.8" H 15300 11750 60  0001 C CNN
+F 3 "" H 15300 11750 60  0000 C CNN
+	5    15300 11750
 	1    0    0    -1
 $EndComp
@@
 F 0 "R2" H 16880 5820 50  0000 L CNN
 F 1 "R_Small" H 16880 5760 50  0000 L CNN
-F 2 "Resistors_SMD:R_0603" H 16850 5800 60  0001 C CNN
+F 2 "Resistors_SMD:R_0603_HandSoldering" H 16850 5800 60  0001 C CNN
 F 3 "" H 16850 5800 60  0000 C CNN
 	1    16850 5800
@@
 F 0 "R3" H 16880 6120 50  0000 L CNN
 F 1 "R_Small" H 16880 6060 50  0000 L CNN
-F 2 "Resistors_SMD:R_0603" H 16850 6100 60  0001 C CNN
+F 2 "Resistors_SMD:R_0603_HandSoldering" H 16850 6100 60  0001 C CNN
 F 3 "" H 16850 6100 60  0000 C CNN
 	1    16850 6100
@@
 Text GLabel 19500 12850 0    60   Input ~ 0
 NRE#
+$Comp
+L Crystal_Small Y1
+U 1 1 5640030C
+P 12550 9550
+F 0 "Y1" H 12550 9650 50  0000 C CNN
+F 1 "Crystal_Small" H 12550 9450 50  0000 C CNN
+F 2 "opendous:Crystal_5x3.2mm" H 12550 9550 60  0001 C CNN
+F 3 "" H 12550 9550 60  0000 C CNN
+	1    12550 9550
+	-1   0    0    1
+$EndComp
+Wire Wire Line
+	13000 9500 12700 9500
+Wire Wire Line
+	12700 9500 12700 9400
+Wire Wire Line
+	12700 9400 12450 9400
+Wire Wire Line
+	12450 9400 12450 9550
+Wire Wire Line
+	13000 9600 12650 9600
+Wire Wire Line
+	12650 9550 12650 9700
+$Comp
+L C_Small C1
+U 1 1 564004B3
+P 12400 9800
+F 0 "C1" H 12410 9870 50  0000 L CNN
+F 1 "C_Small" H 12410 9720 50  0000 L CNN
+F 2 "Capacitors_SMD:C_0603_HandSoldering" H 12400 9800 60  0001 C CNN
+F 3 "" H 12400 9800 60  0000 C CNN
+	1    12400 9800
+	1    0    0    -1
+$EndComp
+$Comp
+L C_Small C2
+U 1 1 56400560
+P 12650 9800
+F 0 "C2" H 12660 9870 50  0000 L CNN
+F 1 "C_Small" H 12660 9720 50  0000 L CNN
+F 2 "Capacitors_SMD:C_0603_HandSoldering" H 12650 9800 60  0001 C CNN
+F 3 "" H 12650 9800 60  0000 C CNN
+	1    12650 9800
+	1    0    0    -1
+$EndComp
+Wire Wire Line
+	12450 9550 12400 9550
+Wire Wire Line
+	12400 9550 12400 9700
+Connection ~ 12650 9600
+$Comp
+L GND #PWR09
+U 1 1 56400687
+P 12400 9950
+F 0 "#PWR09" H 12400 9700 50  0001 C CNN
+F 1 "GND" H 12400 9800 50  0000 C CNN
+F 2 "" H 12400 9950 60  0000 C CNN
+F 3 "" H 12400 9950 60  0000 C CNN
+	1    12400 9950
+	1    0    0    -1
+$EndComp
+$Comp
+L GND #PWR010
+U 1 1 56400704
+P 12650 9950
+F 0 "#PWR010" H 12650 9700 50  0001 C CNN
+F 1 "GND" H 12650 9800 50  0000 C CNN
+F 2 "" H 12650 9950 60  0000 C CNN
+F 3 "" H 12650 9950 60  0000 C CNN
+	1    12650 9950
+	1    0    0    -1
+$EndComp
+Wire Wire Line
+	12400 9900 12400 9950
+Wire Wire Line
+	12650 9900 12650 9950
 $EndSCHEMATC

Commit message: a20 schematics
Parts:
- added C3, C4: C_Small, Capacitors_SMD:C_0603, symbol C_Small
- added R4: R_Small, Resistors_SMD:R_0603, symbol R_Small
- added Y2: Crystal_Small, tinycom:crystal3215, symbol Crystal_Small
- C1, C2: footprint Capacitors_SMD:C_0603_HandSoldering -> Capacitors_SMD:C_0603
- R1, R2, R3: footprint Resistors_SMD:R_0603_HandSoldering -> Resistors_SMD:R_0603
Connections:
- net GND: now also P1.2 (P2), P2.15 (P15), U1.AA18 (GND25_TVIN), U1.G3 (GND_DRAM), U1.G4 (GND_DRAM), U1.J11 (GND), U1.J5 (GND_DRAM), U1.K11 (GND), U1.K12 (GND), U1.K13 (GND), U1.K5 (GND_DRAM), U1.L10 (GND), U1.L11 (GND), U1.L12 (GND), U1.M10 (GND), U1.M11 (GND), U1.M12 (GND), U1.M13 (GND), U1.M14 (GND0_SATA), U1.M9 (GND_DLL), U1.N10 (GND_DLL), U1.N11 (GND), U1.N13 (GND1_SATA), U1.N14 (GND2_SATA), U1.N16 (VDD25_1_SATA), U1.N5 (GND_DRAM), U1.P10 (GND_DLL), U1.P11 (GND), U1.P12 (GND), U1.P15 (PLLGND), U1.P5 (GND_DRAM), U1.R11 (GND), U1.R12 (GND), U1.T11 (GND), U1.T16 (PLLDV), U1.T9 (GND), U1.U19 (AGND), U1.U5 (GND_DRAM), U1.V19 (HPGND), U1.V5 (GND_DRAM), U1.W10 (GND_LVDS), U1.W11 (GND_LVDS), U1.W9 (GND_LVDS), U1.Y18 (GND33_TVIN), U1.Y7 (GND_DRAM), U1.Y8 (GND_DRAM), C3.2, C4.2, R4.2
- net SDC0_D2: now reaches U1.K19 (SDC0_D2/JTAG_CK1/PF5)
- net SDC0_D2: now also P1.15 (P15)
- net SDC0_D3: now reaches U1.K20 (SDC0_D3/UART0_RX/PF4)
- net SDC0_D3: now also P1.13 (P13)
- net SDC0_CMD: now reaches U1.L19 (SDC0_CMD/JTAG_DO1/PF3)
- net SDC0_CMD: now also P1.11 (P11)
- net SDC0_CLK: now reaches U1.L20 (SDC0_CLK/UART0_TX/PF2)
- net SDC0_CLK: now also P1.9 (P9)
- net SDC0_D0: now reaches U1.M19 (SDC0_D0/JTAG_DI1/PF1)
- net SDC0_D0: now also P1.7 (P7)
- net SDC0_D1: now reaches U1.M20 (SDC0_D1/JTAG_MS1/PF0)
- net SDC0_D1: now also P1.5 (P5)
- net at U1.AA7 (SZQ): now also R4.1
- net SVREF: now reaches U1.AA8 (SVREF3)
- net SVREF: now also R2.2, R3.1, U1.H3 (SVREF0), U1.H4 (SVREF1), U1.Y5 (SVREF2), U2.H1 (VREFDQ), U2.M8 (VREFCA)
- net VCC_15: now reaches U1.G5 (VCC_DRAM)
- net VCC_15: now also P1.4 (P4), U1.H5 (VCC_DRAM), U1.L5 (VCC_DRAM), U1.M5 (VCC_DRAM), U1.M8 (VDD_DLL), U1.N9 (VDD_DLL), U1.P9 (VDD_DLL), U1.R5 (VCC_DRAM), U1.T5 (VCC_DRAM), U1.W5 (VCC_DRAM), U1.W6 (VCC_DRAM), U1.W7 (VCC_DRAM), U1.Y6 (VCC_DRAM)
- net at U1.F1 (CLK32K_IN): now also C3.1, Y2.2
- net at U1.F2 (CLK32K_OUT): now also C4.1, Y2.1
- net UDM0: now reaches U1.N20 (DM0)
- net UDM0: now also P1.16 (P16)
- net UDP0: now reaches U1.N21 (DP0)
- net UDP0: now also P1.14 (P14)
- net UDM1: now reaches U1.P20 (DM1)
- net UDM1: now also P1.12 (P12)
- net UDP1: now reaches U1.P21 (DP1)
- net UDP1: now also P1.10 (P10)
- net UDM2: now reaches U1.R20 (DM2)
- net UDM2: now also P2.14 (P14)
- net UDP2: now reaches U1.R21 (DP2)
- net UDP2: now also P2.16 (P16)
- net UART0_TX: now reaches U1.A7 (UART0_TX/IR1_TX/PB22)
- net UART0_TX: now also P1.1 (P1)
- net UART0_RX: now reaches U1.B7 (UART0_RX/IR1_RX/PB23)
- net UART0_RX: now also P1.3 (P3)
- net VCC_12: now reaches P1.6 (P6)
- net VCC_33: now reaches P1.8 (P8)
- net VCC_30: now reaches P2.13 (P13)
- no-connect marks 9 -> 249
Other:
- moved on the sheet: P2

Commit message: a20 schematics
Parts:
- added R5, R6, R7, R? (x2): R_Small, Resistors_SMD:R_0603, symbol R_Small
Connections:
- net GND: now also U1.H16 (TEST), U1.K14 (ULGND), U1.L13 (UGND_T), U1.L14 (UGND_C), U1.T10 (JTAG_SEL), U1.W18 (GND33_TVOUT), U3.13 (VSS), U3.36 (VSS)
- net NRB0: now also R7.2
- net NWE#: now also R6.2
- net VCC_12: now also U1.H11 (VDD_CPU), U1.H12 (VDD_CPU), U1.H13 (VDD_CPU), U1.H14 (VDD_CPU), U1.J13 (VDD_CPU), U1.J15 (VDD_INT), U1.J16 (VDD_INT), U1.K10 (VDD_INT), U1.K15 (VDD_INT), U1.K16 (ULVDD), U1.K9 (VDD_INT), U1.L8 (VDD_INT), U1.L9 (VDD_INT), U1.R10 (VDD_INT), U1.R9 (VDD_INT), U1.T8 (VDD_INT)
- net VCC_30: now also U1.T19 (AVCC)
- net VCC_33: now also U1.AB19 (HPVCCIN), U1.H10 (VCC), U1.H15 (VCC), U1.H19 (VCC_NAND), U1.H8 (VCC), U1.H9 (VCC), U1.J10 (VCC), U1.J14 (VCC), U1.J19 (VCC_NAND), U1.J8 (VCC), U1.J9 (VCC), U1.L15 (UVCC_T), U1.L16 (UVCC_C), U1.N19 (VCC_CARD), U1.W12 (VCC_LVDS), U1.W13 (VCC_LVDS), U1.W14 (VCC_LVDS), U1.W15 (VCC33_TVOUT), U1.W16 (VCC33_TVIN), U3.12 (VCC), U3.37 (VCC), R?.1, R?.1
- net VDD_33: now reaches U1.K8 (RTC_VDD)
- net VDD_12: now reaches U1.M15 (VDD12_0_SATA)
- net VDD_12: now also U1.M16 (VDD12_1_SATA)
- net at U1.C14 (RESET#): now also R?.2
- net at U1.F5 (NMI#): now also R?.2
- net NCE0: now reaches U1.K23 (NCE0/PC4)
- net NCE0: now also U3.9 (CE#)
- net at U3.19 (WP#): now also R5.2
- new net +3V3: R5.1, R6.1, R7.1
- no-connect marks 249 -> 258

Commit message: add capacitors
Parts:
- added C10, C11, C12, C13, C14, C15, C16, C17, C18, C19, C20, C5, C6, C7, C8, C9: C_Small, Capacitors_SMD:C_0603, symbol C_Small
- gave numbers to parts that had none: 2
Connections:
- net GND: now also C10.2, C11.2, C12.2, C13.2, C14.2, C15.2, C16.2, C17.2, C18.2, C19.2, C20.2, C5.2, C6.2, C7.2, C8.2, C9.2
- net VCC_12: now also C13.1, C14.1, C15.1, C20.1, C6.1
- net VCC_15: now also C10.1, C11.1, C12.1, C7.1, C8.1, C9.1
- net VCC_33: now also C16.1, C17.1, C18.1, C19.1, C5.1

Commit message: add routing
Connections:
- net +1V5 is gone; now on net VCC_15: R2.1, U2.A1 (VDDQ), U2.A8 (VDDQ), U2.B2 (VDD), U2.C1 (VDDQ), U2.C9 (VDDQ), U2.D2 (VDDQ), U2.D9 (VDD), U2.E9 (VDDQ), U2.F1 (VDDQ), U2.G7 (VDD), U2.H2 (VDDQ), U2.H9 (VDDQ), U2.K2 (VDD), U2.K8 (VDD), U2.N1 (VDD), U2.N9 (VDD), U2.R1 (VDD), U2.R9 (VDD)
- net +3V3 is gone; now on net VCC_33: R5.1, R6.1, R7.1
- net VDD_33 is gone; now on net VCC_33: U1.K8 (RTC_VDD)
Changed lines of the file:
@@
 $EndComp
 $Comp
-L GND #PWR35
+L GND #PWR01
 U 1 1 563E445F
 P 21050 6550
-F 0 "#PWR35" H 21050 6300 50  0001 C CNN
+F 0 "#PWR01" H 21050 6300 50  0001 C CNN
 F 1 "GND" H 21050 6400 50  0000 C CNN
 F 2 "" H 21050 6550 60  0000 C CNN
@@
 SCK_P
 $Comp
-L GND #PWR26
+L GND #PWR02
 U 1 1 563ECE56
 P 18200 1250
-F 0 "#PWR26" H 18200 1000 50  0001 C CNN
+F 0 "#PWR02" H 18200 1000 50  0001 C CNN
 F 1 "GND" H 18200 1100 50  0000 C CNN
 F 2 "" H 18200 1250 60  0000 C CNN
 F 3 "" H 18200 1250 60  0000 C CNN
 	1    18200 1250
-	1    0    0    -1
-$EndComp
-$Comp
-L +1V5 #PWR30
-U 1 1 563ED4AE
-P 19800 1100
-F 0 "#PWR30" H 19800 950 50  0001 C CNN
-F 1 "+1V5" H 19800 1240 50  0000 C CNN
-F 2 "" H 19800 1100 60  0000 C CNN
-F 3 "" H 19800 1100 60  0000 C CNN
-	1    19800 1100
-	1    0    0    -1
-$EndComp
-$Comp
-L +1V5 #PWR31
-U 1 1 563ED57F
-P 19800 7250
-F 0 "#PWR31" H 19800 7100 50  0001 C CNN
-F 1 "+1V5" H 19800 7390 50  0000 C CNN
-F 2 "" H 19800 7250 60  0000 C CNN
-F 3 "" H 19800 7250 60  0000 C CNN
-	1    19800 7250
-	1    0    0    -1
-$EndComp
-$Comp
-L +1V5 #PWR20
-U 1 1 563EDD3D
-P 16850 5600
-F 0 "#PWR20" H 16850 5450 50  0001 C CNN
-F 1 "+1V5" H 16850 5740 50  0000 C CNN
-F 2 "" H 16850 5600 60  0000 C CNN
-F 3 "" H 16850 5600 60  0000 C CNN
-	1    16850 5600
 	1    0    0    -1
 $EndComp
@@
 $EndComp
 $Comp
-L GND #PWR21
+L GND #PWR03
 U 1 1 563EDF36
 P 16850 6300
-F 0 "#PWR21" H 16850 6050 50  0001 C CNN
+F 0 "#PWR03" H 16850 6050 50  0001 C CNN
 F 1 "GND" H 16850 6150 50  0000 C CNN
 F 2 "" H 16850 6300 60  0000 C CNN
@@
 $EndComp
 $Comp
-L GND #PWR22
+L GND #PWR04
 U 1 1 563EE398
 P 17600 5550
-F 0 "#PWR22" H 17600 5300 50  0001 C CNN
+F 0 "#PWR04" H 17600 5300 50  0001 C CNN
 F 1 "GND" H 17600 5400 50  0000 C CNN
 F 2 "" H 17600 5550 60  0000 C CNN
 F 3 "" H 17600 5550 60  0000 C CNN
 	1    17600 5550
-	1    0    0    -1
-$EndComp
-$Comp
-L +1V5 #PWR23
-U 1 1 563EF32F
-P 17650 2100
-F 0 "#PWR23" H 17650 1950 50  0001 C CNN
-F 1 "+1V5" H 17650 2240 50  0000 C CNN
-F 2 "" H 17650 2100 60  0000 C CNN
-F 3 "" H 17650 2100 60  0000 C CNN
-	1    17650 2100
 	1    0    0    -1
 $EndComp
@@
 $EndComp
 $Comp
-L GND #PWR10
+L GND #PWR05
 U 1 1 56400687
 P 12400 9950
-F 0 "#PWR10" H 12400 9700 50  0001 C CNN
+F 0 "#PWR05" H 12400 9700 50  0001 C CNN
 F 1 "GND" H 12400 9800 50  0000 C CNN
 F 2 "" H 12400 9950 60  0000 C CNN
@@
 $EndComp
 $Comp
-L GND #PWR11
+L GND #PWR06
 U 1 1 56400704
 P 12650 9950
-F 0 "#PWR11" H 12650 9700 50  0001 C CNN
+F 0 "#PWR06" H 12650 9700 50  0001 C CNN
 F 1 "GND" H 12650 9800 50  0000 C CNN
 F 2 "" H 12650 9950 60  0000 C CNN
@@
 $EndComp
 $Comp
-L GND #PWR9
+L GND #PWR07
 U 1 1 56408532
 P 12150 9250
-F 0 "#PWR9" H 12150 9000 50  0001 C CNN
+F 0 "#PWR07" H 12150 9000 50  0001 C CNN
 F 1 "GND" H 12150 9100 50  0000 C CNN
 F 2 "" H 12150 9250 60  0000 C CNN
@@
 $EndComp
 $Comp
-L GND #PWR12
+L GND #PWR08
 U 1 1 56408573
 P 12700 9300
-F 0 "#PWR12" H 12700 9050 50  0001 C CNN
+F 0 "#PWR08" H 12700 9050 50  0001 C CNN
 F 1 "GND" H 12700 9150 50  0000 C CNN
 F 2 "" H 12700 9300 60  0000 C CNN
@@
 $EndComp
 $Comp
-L GND #PWR14
+L GND #PWR09
 U 1 1 5640D8CA
 P 12750 6950
-F 0 "#PWR14" H 12750 6700 50  0001 C CNN
+F 0 "#PWR09" H 12750 6700 50  0001 C CNN
 F 1 "GND" H 12750 6800 50  0000 C CNN
 F 2 "" H 12750 6950 60  0000 C CNN
@@
 $EndComp
 $Comp
-L GND #PWR32
+L GND #PWR010
 U 1 1 56408FCA
 P 19800 9350
-F 0 "#PWR32" H 19800 9100 50  0001 C CNN
+F 0 "#PWR010" H 19800 9100 50  0001 C CNN
 F 1 "GND" H 19800 9200 50  0000 C CNN
 F 2 "" H 19800 9350 60  0000 C CNN
@@
 UDP2
 $Comp
-L GND #PWR33
+L GND #PWR011
 U 1 1 56411561
 P 20650 10200
-F 0 "#PWR33" H 20650 9950 50  0001 C CNN
+F 0 "#PWR011" H 20650 9950 50  0001 C CNN
 F 1 "GND" H 20650 10050 50  0000 C CNN
 F 2 "" H 20650 10200 60  0000 C CNN
@@
 NoConn ~ 7500 6050
 $Comp
-L GND #PWR8
+L GND #PWR012
 U 1 1 56414A5D
 P 8850 1300
-F 0 "#PWR8" H 8850 1050 50  0001 C CNN
+F 0 "#PWR012" H 8850 1050 50  0001 C CNN
 F 1 "GND" H 8850 1150 50  0000 C CNN
 F 2 "" H 8850 1300 60  0000 C CNN
@@
 VCC_15
 $Comp
-L GND #PWR1
+L GND #PWR013
 U 1 1 56417328
 P 800 9350
-F 0 "#PWR1" H 800 9100 50  0001 C CNN
+F 0 "#PWR013" H 800 9100 50  0001 C CNN
 F 1 "GND" H 800 9200 50  0000 C CNN
 F 2 "" H 800 9350 60  0000 C CNN
@@
 NoConn ~ 1050 13300
 $Comp
-L GND #PWR3
+L GND #PWR014
 U 1 1 56417B02
 P 900 13450
-F 0 "#PWR3" H 900 13200 50  0001 C CNN
+F 0 "#PWR014" H 900 13200 50  0001 C CNN
 F 1 "GND" H 900 13300 50  0000 C CNN
 F 2 "" H 900 13450 60  0000 C CNN
@@
 NoConn ~ 1050 13700
 $Comp
-L GND #PWR2
+L GND #PWR015
 U 1 1 56417F5A
 P 850 13800
-F 0 "#PWR2" H 850 13550 50  0001 C CNN
+F 0 "#PWR015" H 850 13550 50  0001 C CNN
 F 1 "GND" H 850 13650 50  0000 C CNN
 F 2 "" H 850 13800 60  0000 C CNN
@@
 NoConn ~ 5650 11400
 $Comp
-L GND #PWR6
+L GND #PWR016
 U 1 1 56418E41
 P 5850 12050
-F 0 "#PWR6" H 5850 11800 50  0001 C CNN
+F 0 "#PWR016" H 5850 11800 50  0001 C CNN
 F 1 "GND" H 5850 11900 50  0000 C CNN
 F 2 "" H 5850 12050 60  0000 C CNN
@@
 $EndComp
 $Comp
-L GND #PWR7
+L GND #PWR017
 U 1 1 56419222
 P 5900 12300
-F 0 "#PWR7" H 5900 12050 50  0001 C CNN
+F 0 "#PWR017" H 5900 12050 50  0001 C CNN
 F 1 "GND" H 5900 12150 50  0000 C CNN
 F 2 "" H 5900 12300 60  0000 C CNN
@@
 NoConn ~ 11650 14450
 $Comp
-L GND #PWR16
+L GND #PWR018
 U 1 1 5641B53D
 P 12900 9850
-F 0 "#PWR16" H 12900 9600 50  0001 C CNN
+F 0 "#PWR018" H 12900 9600 50  0001 C CNN
 F 1 "GND" H 12900 9700 50  0000 C CNN
 F 2 "" H 12900 9850 60  0000 C CNN
@@
 NoConn ~ 13000 10700
 $Comp
-L GND #PWR15
+L GND #PWR019
 U 1 1 5641BA06
 P 12850 11350
-F 0 "#PWR15" H 12850 11100 50  0001 C CNN
+F 0 "#PWR019" H 12850 11100 50  0001 C CNN
 F 1 "GND" H 12850 11200 50  0000 C CNN
 F 2 "" H 12850 11350 60  0000 C CNN
@@
 NoConn ~ 13000 12600
 $Comp
-L GND #PWR13
+L GND #PWR020
 U 1 1 5641C0BF
 P 12700 12700
-F 0 "#PWR13" H 12700 12450 50  0001 C CNN
+F 0 "#PWR020" H 12700 12450 50  0001 C CNN
 F 1 "GND" H 12700 12550 50  0000 C CNN
 F 2 "" H 12700 12700 60  0000 C CNN
@@
 $EndComp
 $Comp
-L GND #PWR24
+L GND #PWR021
 U 1 1 5641C64B
 P 17750 14500
-F 0 "#PWR24" H 17750 14250 50  0001 C CNN
+F 0 "#PWR021" H 17750 14250 50  0001 C CNN
 F 1 "GND" H 17750 14350 50  0000 C CNN
 F 2 "" H 17750 14500 60  0000 C CNN
@@
 $EndComp
 $Comp
-L GND #PWR25
+L GND #PWR022
 U 1 1 5641CC6D
 P 17800 13850
-F 0 "#PWR25" H 17800 13600 50  0001 C CNN
+F 0 "#PWR022" H 17800 13600 50  0001 C CNN
 F 1 "GND" H 17800 13700 50  0000 C CNN
 F 2 "" H 17800 13850 60  0000 C CNN
@@
 VCC_33
 Text GLabel 12950 8550 0    60   Input ~ 0
-VDD_33
-$Comp
-L GND #PWR34
+VCC_33
+$Comp
+L GND #PWR023
 U 1 1 5643044F
 P 20800 13600
-F 0 "#PWR34" H 20800 13350 50  0001 C CNN
+F 0 "#PWR023" H 20800 13350 50  0001 C CNN
 F 1 "GND" H 20800 13450 50  0000 C CNN
 F 2 "" H 20800 13600 60  0000 C CNN
@@
 $EndComp
 $Comp
-L +3.3V #PWR29
-U 1 1 56431B98
-P 18750 12950
-F 0 "#PWR29" H 18750 12800 50  0001 C CNN
-F 1 "+3.3V" H 18750 13090 50  0000 C CNN
-F 2 "" H 18750 12950 60  0000 C CNN
-F 3 "" H 18750 12950 60  0000 C CNN
-	1    18750 12950
-	1    0    0    -1
-$EndComp
-$Comp
 L R_Small R6
 U 1 1 5643228C
@@
 $EndComp
 $Comp
-L +3.3V #PWR27
-U 1 1 56432293
-P 18500 12400
-F 0 "#PWR27" H 18500 12250 50  0001 C CNN
-F 1 "+3.3V" H 18500 12540 50  0000 C CNN
-F 2 "" H 18500 12400 60  0000 C CNN
-F 3 "" H 18500 12400 60  0000 C CNN
-	1    18500 12400
-	1    0    0    -1
-$EndComp
-$Comp
 L R_Small R7
 U 1 1 564328C3
@@
 F 3 "" H 18750 12350 60  0000 C CNN
 	1    18750 12350
-	1    0    0    -1
-$EndComp
-$Comp
-L +3.3V #PWR28
-U 1 1 564328C9
-P 18750 12150
-F 0 "#PWR28" H 18750 12000 50  0001 C CNN
-F 1 "+3.3V" H 18750 12290 50  0000 C CNN
-F 2 "" H 18750 12150 60  0000 C CNN
-F 3 "" H 18750 12150 60  0000 C CNN
-	1    18750 12150
 	1    0    0    -1
 $EndComp
@@
 VCC_33
 $Comp
-L GND #PWR5
+L GND #PWR025
 U 1 1 5643A4FE
 P 5850 10900
-F 0 "#PWR5" H 5850 10650 50  0001 C CNN
+F 0 "#PWR025" H 5850 10650 50  0001 C CNN
 F 1 "GND" H 5850 10750 50  0000 C CNN
 F 2 "" H 5850 10900 60  0000 C CNN
@@
 NoConn ~ 1050 14100
 $Comp
-L GND #PWR4
+L GND #PWR026
 U 1 1 5643BDD7
 P 950 11000
-F 0 "#PWR4" H 950 10750 50  0001 C CNN
+F 0 "#PWR026" H 950 10750 50  0001 C CNN
 F 1 "GND" H 950 10850 50  0000 C CNN
 F 2 "" H 950 11000 60  0000 C CNN
@@
 VCC_33
 $Comp
-L GND #PWR17
+L GND #PWR027
 U 1 1 56440C85
 P 13650 7250
-F 0 "#PWR17" H 13650 7000 50  0001 C CNN
+F 0 "#PWR027" H 13650 7000 50  0001 C CNN
 F 1 "GND" H 13650 7100 50  0000 C CNN
 F 2 "" H 13650 7250 60  0000 C CNN
@@
 $EndComp
 $Comp
-L GND #PWR18
+L GND #PWR028
 U 1 1 56441E51
 P 14450 7250
-F 0 "#PWR18" H 14450 7000 50  0001 C CNN
+F 0 "#PWR028" H 14450 7000 50  0001 C CNN
 F 1 "GND" H 14450 7100 50  0000 C CNN
 F 2 "" H 14450 7250 60  0000 C CNN
@@
 $EndComp
 $Comp
-L GND #PWR19
+L GND #PWR029
 U 1 1 564426D1
 P 15100 7250
-F 0 "#PWR19" H 15100 7000 50  0001 C CNN
+F 0 "#PWR029" H 15100 7000 50  0001 C CNN
 F 1 "GND" H 15100 7100 50  0000 C CNN
 F 2 "" H 15100 7250 60  0000 C CNN
@@
 	14050 7150 14050 7100
 Connection ~ 14200 7150
+Text GLabel 17650 2100 0    60   Input ~ 0
+VCC_15
+Text GLabel 19800 1100 2    60   Input ~ 0
+VCC_15
+Text GLabel 16850 5600 0    60   Input ~ 0
+VCC_15
+Text GLabel 18750 12150 0    60   Input ~ 0
+VCC_33
+Text GLabel 18500 12400 0    60   Input ~ 0
+VCC_33
+Text GLabel 19800 7250 2    60   Input ~ 0
+VCC_15
+Text GLabel 18750 12950 0    60   Input ~ 0
+VCC_33
 $EndSCHEMATC
