File: tinycom-a20/tinycom-a20.kicad_pcb (KiCad board)
At the start: 4 copper layers, 40.4 x 41.9 mm, 39 parts, among them P1 CONN_02X08, P2 CONN_02X08, P3 CONN_01X01, U1 ALLWINNERA10/TFBGA441, U2 H5TQG63BFR/FBGA96, U3 H27UBG8T2A/TSOP48, Y1 Crystal_Small, Y2 Crystal_Small

Commit message: delete tracks
Parts:
- removed P1, P2: CONN_02X08, Socket_Strips:Socket_Strip_Straight_2x08
- removed R5, R6, R7: R_Small, Resistors_SMD:R_0603
- removed U3: H27UBG8T2A/TSOP48, tsop48:TSOP48
Routing:
- net VCC_33: track 213.6 -> 0.00 mm, vias 17 -> 0
- net GND: track 120.6 -> 0.00 mm, vias 50 -> 0
- net UART0_RX: track 65.3 -> 0.00 mm
- net UART0_TX: track 53.6 -> 0.00 mm, vias 1 -> 0
- net VCC_15: track 51.8 -> 0.00 mm, vias 30 -> 0
- net VCC_12: track 49.3 -> 0.00 mm, vias 7 -> 0
- net SDC0_D1: track 32.7 -> 0.00 mm
- net UDP2: track 31.3 -> 0.00 mm, vias 1 -> 0
- net UDP1: track 30.6 -> 0.00 mm
- net SDC0_CLK: track 29.3 -> 0.00 mm, vias 1 -> 0
- net UDP0: track 28.7 -> 0.00 mm
- net SDC0_D0: track 27.9 -> 0.00 mm, vias 2 -> 0
- net NWE#: track 27.7 -> 0.00 mm, vias 3 -> 0
- net UDM2: track 27.6 -> 0.00 mm, vias 1 -> 0
- net VCC_30: track 27.1 -> 0.00 mm, vias 1 -> 0
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
Commit message: xxx
Parts:
- added P1: CONN_02X10, Pin_Headers:Pin_Header_Straight_2x10, F.Cu at (93.2, 160.2)
- added P2: CONN_02X10, Pin_Headers:Pin_Header_Straight_2x10, F.Cu at (93.4, 124.9)
Connections:
- U1 pad G20: ND7 -> (no net)
- U1 pad G21: ND6 -> (no net)
- U1 pad G22: ND3 -> (no net)
- U1 pad G23: ND2 -> (no net)
- U1 pad H20: ND5 -> (no net)
- U1 pad H21: ND4 -> (no net)
- U1 pad H22: ND1 -> (no net)
- U1 pad H23: ND0 -> (no net)
- U1 pad J23: NRB0 -> (no net)
- U1 pad K22: NRE# -> (no net)
- U1 pad K23: NCE0 -> (no net)
- U1 pad L23: NCLE -> (no net)
- U1 pad M22: NALE -> (no net)
- U1 pad M23: NWE# -> (no net)

Commit message: improve placement
Parts:
- P1, P2: moved to B.Cu
- R1, R4: value R_Small -> 330R
- R2, R3: value R_Small -> 2K
- moved C2 18.8 mm to (123.4, 144.4), turned to 270 degrees
- moved C5 17.6 mm to (119.6, 129.2), turned to 90 degrees
- moved C6 16.4 mm to (117.9, 129.2), turned to 90 degrees
- moved Y1 12.5 mm to (124.3, 140.2), turned to 90 degrees
- moved C14 11.4 mm to (123.5, 132.8), turned to 90 degrees
- moved C22 10.2 mm to (113.8, 151.8)
- moved C1 7.32 mm to (123.5, 135.9), turned to 90 degrees
- moved C21 7.27 mm to (112.1, 151.8)
- moved C4 6.69 mm to (102.4, 131.3)
- moved C3 6.06 mm to (100.7, 131.3)
- moved C19 4.07 mm to (107.2, 129.2)
- moved Y2 3.14 mm to (104.5, 134.7), turned to 270 degrees
- moved R4 3.11 mm to (110.4, 151.7)
- moved P1 2.76 mm to (93.9, 157.6), turned to 270 degrees
- moved P2 2.49 mm to (93.9, 122.5), turned to 270 degrees
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Routing:
- net Net-(C2-Pad1): track 26.6 -> 0.00 mm
- net Net-(C1-Pad1): track 17.7 -> 0.00 mm
- net Net-(C4-Pad1): track 11.1 -> 5.72 mm
- net Net-(C3-Pad1): track 11.3 -> 6.61 mm
- net Net-(R4-Pad1): track 7.10 -> 4.29 mm
- net RESET#: track 4.45 -> 3.50 mm
- net SVREF: track 48.8 -> 49.3 mm
- net (no net): vias 97 -> 77
Other:
- board size 40.4 x 41.9 mm -> 41.3 x 41.9 mm

Commit message: a20 layout
Routing:
- removed copper zone on In1.Cu, net GND
- removed copper zone on In2.Cu, net VCC_12
- removed copper zone on In2.Cu, net VCC_15
Other:
- board size 41.3 x 41.9 mm -> 41.4 x 40.9 mm
Changed lines of the file:
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@@
     (links 270)
     (no_connects 206)
-    (area 83.860999 120.066999 125.297001 162.127001)
+    (area 84.424999 120.824999 125.975001 161.875001)
     (thickness 1.6)
     (drawings 18)
-    (tracks 1403)
+    (tracks 1404)
     (zones 0)
     (modules 35)
@@
     )
   )
+  (gr_line (start 118.2 154) (end 125.9 154) (layer Edge.Cuts) (width 0.15))
+  (gr_line (start 118.2 161.8) (end 118.2 154) (layer Edge.Cuts) (width 0.15))
+  (gr_line (start 92 161.8) (end 92.2 161.8) (layer Edge.Cuts) (width 0.15))
+  (gr_line (start 92 154.3) (end 92 161.8) (layer Edge.Cuts) (width 0.15))
+  (gr_line (start 84.5 154.3) (end 92 154.3) (layer Edge.Cuts) (width 0.15))
+  (gr_line (start 84.5 127.9) (end 84.5 154.3) (layer Edge.Cuts) (width 0.15))
+  (gr_line (start 125.9 154) (end 125.9 127.8) (layer Edge.Cuts) (width 0.15))
+  (gr_line (start 92 127.9) (end 84.5 127.9) (layer Edge.Cuts) (width 0.15))
+  (gr_line (start 92 120.9) (end 92 127.9) (layer Edge.Cuts) (width 0.15))
+  (gr_line (start 118.3 120.9) (end 92 120.9) (layer Edge.Cuts) (width 0.15))
+  (gr_line (start 118.3 127.8) (end 118.3 120.9) (layer Edge.Cuts) (width 0.15))
+  (gr_line (start 118.6 127.8) (end 118.3 127.8) (layer Edge.Cuts) (width 0.15))
+  (gr_line (start 125.9 127.8) (end 118.6 127.8) (layer Edge.Cuts) (width 0.15))
+  (gr_line (start 92.2 161.8) (end 118.2 161.8) (layer Edge.Cuts) (width 0.15))
   (gr_text http://tinycom.org/ (at 107.3675 140.624 90) (layer B.SilkS)
     (effects (font (size 1.5 1.5) (thickness 0.3)) (justify mirror))
@@
     (effects (font (size 4 4) (thickness 0.5)) (justify mirror))
   )
-  (gr_line (start 92.964 120.142) (end 93.472 120.142) (layer Edge.Cuts) (width 0.15))
-  (gr_line (start 92.964 122.936) (end 92.964 120.142) (layer Edge.Cuts) (width 0.15))
   (gr_line (start 92.964 122.936) (end 92.964 122.936) (layer Edge.Cuts) (width 0.15))
-  (gr_line (start 92.964 127.762) (end 92.964 122.936) (layer Edge.Cuts) (width 0.15))
-  (gr_line (start 83.936 127.162) (end 92.064 127.162) (layer Edge.Cuts) (width 0.15))
-  (gr_line (start 84.836 154.94) (end 84.836 127.762) (layer Edge.Cuts) (width 0.15))
-  (gr_line (start 92.826 154.34) (end 83.936 154.34) (layer Edge.Cuts) (width 0.15))
-  (gr_line (start 93.726 162.052) (end 93.726 154.94) (layer Edge.Cuts) (width 0.15))
-  (gr_line (start 116.078 162.052) (end 93.726 162.052) (layer Edge.Cuts) (width 0.15))
-  (gr_line (start 116.078 154.686) (end 116.078 162.052) (layer Edge.Cuts) (width 0.15))
-  (gr_line (start 124.322 154.086) (end 115.178 154.086) (layer Edge.Cuts) (width 0.15))
-  (gr_line (start 125.222 127.508) (end 125.222 154.686) (layer Edge.Cuts) (width 0.15))
-  (gr_line (start 114.67 126.908) (end 124.322 126.908) (layer Edge.Cuts) (width 0.15))
-  (gr_line (start 115.57 120.142) (end 115.57 127.508) (layer Edge.Cuts) (width 0.15))
-  (gr_line (start 93.472 120.142) (end 115.57 120.142) (layer Edge.Cuts) (width 0.15))
+  (segment (start 92 162.1) (end 91.9 162.1) (width 0.15) (layer Dwgs.User) (net 0))
   (via (at 109.601 156.1592) (size 0.6) (drill 0.3) (layers F.Cu B.Cu) (net 0))
   (via (at 111.95728 145.55922) (size 0.6) (drill 0.3) (layers F.Cu B.Cu) (net 0))
@@
   (segment (start 103.948898 134.45) (end 103.6 134.101102) (width 0.15) (layer F.Cu) (net 62))
   (segment (start 103.6 131.0578) (end 104.0128 130.645) (width 0.15) (layer F.Cu) (net 62))
-  (zone (net 23) (net_name GND) (layer In1.Cu) (hatch edge 0.508)
-    (connect_pads (clearance 0.1))
-    (min_thickness 0.254)
-    (fill yes (arc_segments 16) (thermal_gap 0.508) (thermal_bridge_width 0.508))
-    (polygon
-      (pts
-        (xy 93.0275 120.142) (xy 115.6335 120.142) (xy 115.6335 127.508) (xy 125.2855 127.508) (xy 125.2855 154.686)
-        (xy 116.078 154.686) (xy 116.078 162.052) (xy 93.7895 162.052) (xy 93.7895 154.94) (xy 84.8995 154.94)
-        (xy 84.8995 127.762) (xy 93.0275 127.762)
-      )
-    )
-  )
-  (zone (net 57) (net_name VCC_15) (layer In2.Cu) (hatch edge 0.508)
-    (connect_pads (clearance 0.1))
-    (min_thickness 0.254)
-    (fill yes (arc_segments 16) (thermal_gap 0.508) (thermal_bridge_width 0.508))
-    (polygon
-      (pts
-        (xy 83.9995 127.162) (xy 108.6248 127.035) (xy 108.6248 154.213) (xy 83.9995 154.34)
-      )
-    )
-  )
-  (zone (net 58) (net_name VCC_12) (layer In2.Cu) (hatch edge 0.508)
-    (connect_pads (clearance 0.1))
-    (min_thickness 0.254)
-    (fill yes (arc_segments 16) (thermal_gap 0.508) (thermal_bridge_width 0.508))
-    (polygon
-      (pts
-        (xy 109.1328 127.035) (xy 124.3728 127.035) (xy 124.3855 154.086) (xy 109.1328 154.213)
-      )
-    )
-  )
 )

Commit message: before resize vias
Connections:
- P1 pad 10: UDP1 -> UD1_N
- P1 pad 12: UDM1 -> UD1_P
- P1 pad 14: UDP2 -> UD2_N
- P1 pad 16: UDM2 -> UD2_P
- P1 pad 6: UDP0 -> UD0_N
- P1 pad 8: UDM0 -> UD0_P
- P2 pad 10: SDC0_D0 -> SDC0_D1
- P2 pad 12: SDC0_D1 -> SDC0_D0
- P2 pad 14: (no net) -> SDC0_CLK
- P2 pad 15: UART0_TX -> UART0_RX
- P2 pad 16: (no net) -> SDC0_CMD
- P2 pad 17: UART0_RX -> UART0_TX
- P2 pad 18: (no net) -> SDC0_D3
- P2 pad 2: SDC0_D2 -> (no net)
- P2 pad 20: (no net) -> SDC0_D2
- P2 pad 4: SDC0_D3 -> (no net)
- P2 pad 6: SDC0_CMD -> (no net)
- P2 pad 8: SDC0_CLK -> (no net)
- U1 pad N20: UDM0 -> UD0_N
- U1 pad N21: UDP0 -> UD0_P
- U1 pad P20: UDM1 -> UD1_N
- U1 pad P21: UDP1 -> UD1_P
- U1 pad R20: UDM2 -> UD2_N
- U1 pad R21: UDP2 -> UD2_P
Routing:
- net UD0_P: track 0.00 -> 31.1 mm, vias 0 -> 1
- net UD0_N: track 0.00 -> 30.7 mm, vias 0 -> 1
- net SDC0_D1: track 0.00 -> 27.8 mm, vias 0 -> 1
- net UD1_P: track 0.00 -> 26.0 mm, vias 0 -> 1
- net UD1_N: track 0.00 -> 25.0 mm, vias 0 -> 1
- net SDC0_D0: track 0.00 -> 24.0 mm, vias 0 -> 1
- net SDC0_CLK: track 0.00 -> 22.8 mm, vias 0 -> 1
- net UD2_P: track 0.00 -> 22.3 mm, vias 0 -> 1
- net UD2_N: track 0.00 -> 21.9 mm, vias 0 -> 1
- net SDC0_CMD: track 0.00 -> 18.7 mm, vias 0 -> 1
- net SDC0_D3: track 0.00 -> 17.2 mm, vias 0 -> 1
- net SDC0_D2: track 0.00 -> 14.6 mm, vias 0 -> 1
- net UART0_RX: track 0.00 -> 11.5 mm
- net UART0_TX: track 0.00 -> 11.4 mm
- net (no net): vias 77 -> 67
Other:
- net class Default: clearance 0.11 -> 0.15; via_dia 0.6 -> 0.5
- net class Ground: clearance 0.11 -> 0.15; via_dia 0.6 -> 0.5
- net class Power: clearance 0.11 -> 0.15; via_dia 0.6 -> 0.5
- rule trace_clearance: 0.11 -> 0.15

Commit message: check
Connections:
- U1 pad J12: (no net) -> VCC_12
- U1 pad N12: (no net) -> GND
- U1 pad N16: GND -> (no net)
- U1 pad P13: (no net) -> GND
- U1 pad P14: (no net) -> GND
- U1 pad P16: (no net) -> VCC_33
- U1 pad R13: (no net) -> GND
- U1 pad T12: (no net) -> GND
- U1 pad T13: (no net) -> VCC_33
- U1 pad T16: GND -> (no net)
Routing:
- net GND: track 0.00 -> 56.8 mm, vias 0 -> 12
- net VCC_12: track 0.00 -> 23.0 mm, vias 0 -> 1
- net VCC_33: track 0.00 -> 13.6 mm, vias 0 -> 5
- net VCC_15: track 0.00 -> 6.40 mm, vias 0 -> 6
- net Net-(C1-Pad1): track 0.00 -> 6.01 mm
- net Net-(C2-Pad1): track 0.00 -> 5.79 mm
- net (no net): vias 67 -> 48
- added copper zone on In1.Cu, net GND
- added copper zone on In2.Cu, net VCC_15
- added copper zone on In2.Cu, net VCC_33

Commit message: before reroute ddr3
Connections:
- U1 pad J12: VCC_12 -> (no net)
- U1 pad R3: (no net) -> SA14
- U2 pad T7: (no net) -> SA14
Routing:
- net VCC_33: track 13.6 -> 18.1 mm, vias 5 -> 7
- net GND: track 56.8 -> 60.1 mm, vias 12 -> 14
- net SDQ6: track 27.3 -> 26.0 mm
- net UBOOT_SEL: track 11.1 -> 10.3 mm
- net (no net): vias 48 -> 46

Commit message: route ddr data
Parts:
- moved P3 4.78 mm to (112.8, 154.6)
- moved C12 2.69 mm to (92.9, 154.8)
- moved C11 1.80 mm to (99.3, 154.6)
- moved C13 1.72 mm to (95.7, 154.6)
- moved R4 1.18 mm to (111.6, 152.0)
Routing:
- net SRST: track 38.3 -> 0.00 mm
- net SA6: track 34.9 -> 0.00 mm, vias 2 -> 0
- net SA0: track 31.6 -> 0.00 mm, vias 2 -> 0
- net SA8: track 31.1 -> 0.00 mm, vias 2 -> 0
- net SA2: track 31.0 -> 0.00 mm, vias 2 -> 0
- net SODT0: track 29.5 -> 0.00 mm, vias 2 -> 0
- net SA5: track 27.5 -> 0.00 mm, vias 3 -> 0
- net SA4: track 27.3 -> 0.00 mm
- net SA12: track 27.2 -> 0.00 mm, vias 2 -> 0
- net SA10: track 27.0 -> 0.00 mm, vias 2 -> 0
- net SA3: track 25.7 -> 0.00 mm, vias 2 -> 0
- net SA9: track 25.3 -> 0.00 mm
- net SA13: track 24.5 -> 0.00 mm, vias 2 -> 0
- net SA1: track 24.2 -> 0.00 mm, vias 2 -> 0
- net SA11: track 22.9 -> 0.00 mm, vias 2 -> 0
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