File: tinycom-a13/tinycom-a13.sch (KiCad schematic (older format))
At the start: 23 parts, among them P1 CONN_02X08, P2 CONN_02X08, U1 IC_A13, U2 H5TQ2G83BFR/FBGA82, Y1 Crystal

Commit message: change connectors
Parts:
- removed P1, P2: CONN_02X08, Pin_Headers:Pin_Header_Straight_2x08, symbol CONN_02X08
- added P1, P2: CONN_02X10, Pin_Headers:Pin_Header_Straight_2x10, symbol CONN_02X10
Changed lines of the file:
@@
 LIBS:opendous
 LIBS:calculator
-LIBS:tinycom-cpu-cache
 EELAYER 25 0
 EELAYER END
@@
 Text GLabel 10900 3850 2    60   Input ~ 0
 DDR3_D15
-$Comp
-L CONN_02X08 P1
-U 1 1 5623B033
-P 13450 9600
-F 0 "P1" H 13450 10050 50  0000 C CNN
-F 1 "CONN_02X08" V 13450 9600 50  0000 C CNN
-F 2 "Pin_Headers:Pin_Header_Straight_2x08" H 13450 8400 60  0001 C CNN
-F 3 "" H 13450 8400 60  0000 C CNN
-	1    13450 9600
-	1    0    0    -1
-$EndComp
-$Comp
-L CONN_02X08 P2
-U 1 1 5623B4E2
-P 15000 9600
-F 0 "P2" H 15000 10050 50  0000 C CNN
-F 1 "CONN_02X08" V 15000 9600 50  0000 C CNN
-F 2 "Pin_Headers:Pin_Header_Straight_2x08" H 15000 8400 60  0001 C CNN
-F 3 "" H 15000 8400 60  0000 C CNN
-	1    15000 9600
-	1    0    0    -1
-$EndComp
 Text GLabel 10900 11450 2    60   Input ~ 0
 SDC0_D1
@@
 Text GLabel 7500 7650 0    60   Input ~ 0
 UDM0
-Text GLabel 13200 9250 0    60   Input ~ 0
-SDC0_D2
-Text GLabel 13200 9350 0    60   Input ~ 0
-SDC0_D3
-Text GLabel 13200 9450 0    60   Input ~ 0
-SDC0_CMD
-Text GLabel 13200 9550 0    60   Input ~ 0
-SDC0_CLK
-Text GLabel 13200 9650 0    60   Input ~ 0
-SDC0_D0
-Text GLabel 13200 9750 0    60   Input ~ 0
-SDC0_D1
-Text GLabel 13700 9250 2    60   Input ~ 0
-UDM0
-Text GLabel 13700 9350 2    60   Input ~ 0
-UDP0
-Text GLabel 13700 9450 2    60   Input ~ 0
-UDM1
-Text GLabel 13700 9550 2    60   Input ~ 0
-UDP1
-Text GLabel 14750 9250 0    60   Input ~ 0
-CSI_CLK
-Text GLabel 14750 9350 0    60   Input ~ 0
-CSI_MCLK
-Text GLabel 14750 9450 0    60   Input ~ 0
-CSI_HSYNC
-Text GLabel 14750 9550 0    60   Input ~ 0
-CSI_VSYNC
-Text GLabel 14750 9650 0    60   Input ~ 0
-CSI_D0
-Text GLabel 14750 9750 0    60   Input ~ 0
-CSI_D1
-Text GLabel 14750 9850 0    60   Input ~ 0
-CSI_D2
-Text GLabel 14750 9950 0    60   Input ~ 0
-CSI_D3
-Text GLabel 15250 9250 2    60   Input ~ 0
-CSI_D4
-Text GLabel 15250 9350 2    60   Input ~ 0
-CSI_D5
-Text GLabel 15250 9450 2    60   Input ~ 0
-CSI_D6
-Text GLabel 15250 9550 2    60   Input ~ 0
-CSI_D7
-Text GLabel 13200 9850 0    60   Input ~ 0
-UART1_RX
-Text GLabel 13200 9950 0    60   Input ~ 0
-UART1_TX
-Text GLabel 15250 9950 2    60   Input ~ 0
-GND
-Text GLabel 13700 9950 2    60   Input ~ 0
-GND
-Text GLabel 13700 9850 2    60   Input ~ 0
-VCC_15
-Text GLabel 13700 9750 2    60   Input ~ 0
-VCC_14
-Text GLabel 13700 9650 2    60   Input ~ 0
-VCC_33
-Text GLabel 15250 9850 2    60   Input ~ 0
-VCC_30
-Text GLabel 15250 9750 2    60   Input ~ 0
-GND
-Text GLabel 15250 9650 2    60   Input ~ 0
-MICIN1
 Text GLabel 7400 2200 0    60   Input ~ 0
 VCC_33
@@
 $EndComp
 $Comp
-L GND #PWR01
+L GND #PWR2
 U 1 1 5624C74D
 P 6400 5750
-F 0 "#PWR01" H 6400 5500 50  0001 C CNN
+F 0 "#PWR2" H 6400 5500 50  0001 C CNN
 F 1 "GND" H 6400 5600 50  0000 C CNN
 F 2 "" H 6400 5750 60  0000 C CNN
@@
 $EndComp
 $Comp
-L GND #PWR02
+L GND #PWR3
 U 1 1 5624C778
 P 6400 6050
-F 0 "#PWR02" H 6400 5800 50  0001 C CNN
+F 0 "#PWR3" H 6400 5800 50  0001 C CNN
 F 1 "GND" H 6400 5900 50  0000 C CNN
 F 2 "" H 6400 6050 60  0000 C CNN
@@
 VCC_14
 $Comp
-L +3.3V #PWR03
+L +3.3V #PWR7
 U 1 1 5624CB40
 P 7400 2200
-F 0 "#PWR03" H 7400 2050 50  0001 C CNN
+F 0 "#PWR7" H 7400 2050 50  0001 C CNN
 F 1 "+3.3V" H 7400 2340 50  0000 C CNN
 F 2 "" H 7400 2200 60  0000 C CNN
@@
 $EndComp
 $Comp
-L +1V5 #PWR04
+L +1V5 #PWR1
 U 1 1 5624CB62
 P 5250 2150
-F 0 "#PWR04" H 5250 2000 50  0001 C CNN
+F 0 "#PWR1" H 5250 2000 50  0001 C CNN
 F 1 "+1V5" H 5250 2290 50  0000 C CNN
 F 2 "" H 5250 2150 60  0000 C CNN
@@
 DDR3_BA2
 $Comp
-L +1V5 #PWR05
+L +1V5 #PWR14
 U 1 1 5625F72C
 P 15200 3600
-F 0 "#PWR05" H 15200 3450 50  0001 C CNN
+F 0 "#PWR14" H 15200 3450 50  0001 C CNN
 F 1 "+1V5" H 15200 3740 50  0000 C CNN
 F 2 "" H 15200 3600 60  0000 C CNN
@@
 $EndComp
 $Comp
-L GND #PWR06
+L GND #PWR15
 U 1 1 5625F96A
 P 15350 7200
-F 0 "#PWR06" H 15350 6950 50  0001 C CNN
+F 0 "#PWR15" H 15350 6950 50  0001 C CNN
 F 1 "GND" H 15350 7050 50  0000 C CNN
 F 2 "" H 15350 7200 60  0000 C CNN
@@
 DDR3_RST
 $Comp
-L GND #PWR07
+L GND #PWR9
 U 1 1 5625FBB8
 P 11800 5950
-F 0 "#PWR07" H 11800 5700 50  0001 C CNN
+F 0 "#PWR9" H 11800 5700 50  0001 C CNN
 F 1 "GND" H 11800 5800 50  0000 C CNN
 F 2 "" H 11800 5950 60  0000 C CNN
@@
 $EndComp
 $Comp
-L +1V5 #PWR08
+L +1V5 #PWR10
 U 1 1 5625FE07
 P 12000 7100
-F 0 "#PWR08" H 12000 6950 50  0001 C CNN
+F 0 "#PWR10" H 12000 6950 50  0001 C CNN
 F 1 "+1V5" H 12000 7240 50  0000 C CNN
 F 2 "" H 12000 7100 60  0000 C CNN
@@
 $EndComp
 $Comp
-L GND #PWR09
+L GND #PWR11
 U 1 1 5625FF1B
 P 12000 7850
-F 0 "#PWR09" H 12000 7600 50  0001 C CNN
+F 0 "#PWR11" H 12000 7600 50  0001 C CNN
 F 1 "GND" H 12000 7700 50  0000 C CNN
 F 2 "" H 12000 7850 60  0000 C CNN
@@
 $EndComp
 $Comp
-L GND #PWR010
+L GND #PWR12
 U 1 1 56260662
 P 12250 8100
-F 0 "#PWR010" H 12250 7850 50  0001 C CNN
+F 0 "#PWR12" H 12250 7850 50  0001 C CNN
 F 1 "GND" H 12250 7950 50  0000 C CNN
 F 2 "" H 12250 8100 60  0000 C CNN
@@
 NoConn ~ 15100 7350
 $Comp
-L GND #PWR011
+L GND #PWR13
 U 1 1 56261679
 P 12450 7900
-F 0 "#PWR011" H 12450 7650 50  0001 C CNN
+F 0 "#PWR13" H 12450 7650 50  0001 C CNN
 F 1 "GND" H 12450 7750 50  0000 C CNN
 F 2 "" H 12450 7900 60  0000 C CNN
@@
 $EndComp
 $Comp
-L GND #PWR012
+L GND #PWR8
 U 1 1 56262D84
 P 11100 7950
-F 0 "#PWR012" H 11100 7700 50  0001 C CNN
+F 0 "#PWR8" H 11100 7700 50  0001 C CNN
 F 1 "GND" H 11100 7800 50  0000 C CNN
 F 2 "" H 11100 7950 60  0000 C CNN
@@
 $EndComp
 $Comp
-L +1V5 #PWR013
+L +1V5 #PWR16
 U 1 1 562642D9
 P 16050 3500
-F 0 "#PWR013" H 16050 3350 50  0001 C CNN
+F 0 "#PWR16" H 16050 3350 50  0001 C CNN
 F 1 "+1V5" H 16050 3640 50  0000 C CNN
 F 2 "" H 16050 3500 60  0000 C CNN
@@
 $EndComp
 $Comp
-L GND #PWR014
+L GND #PWR17
 U 1 1 562643A7
 P 16100 3900
-F 0 "#PWR014" H 16100 3650 50  0001 C CNN
+F 0 "#PWR17" H 16100 3650 50  0001 C CNN
 F 1 "GND" H 16100 3750 50  0000 C CNN
 F 2 "" H 16100 3900 60  0000 C CNN
@@
 $EndComp
 $Comp
-L GND #PWR015
+L GND #PWR4
 U 1 1 56265943
 P 6850 3500
-F 0 "#PWR015" H 6850 3250 50  0001 C CNN
+F 0 "#PWR4" H 6850 3250 50  0001 C CNN
 F 1 "GND" H 6850 3350 50  0000 C CNN
 F 2 "" H 6850 3500 60  0000 C CNN
@@
 $EndComp
 $Comp
-L GND #PWR016
+L GND #PWR5
 U 1 1 56265988
 P 7050 2700
-F 0 "#PWR016" H 7050 2450 50  0001 C CNN
+F 0 "#PWR5" H 7050 2450 50  0001 C CNN
 F 1 "GND" H 7050 2550 50  0000 C CNN
 F 2 "" H 7050 2700 60  0000 C CNN
@@
 SVREF
 $Comp
-L GND #PWR017
+L GND #PWR6
 U 1 1 562A3A06
 P 7100 5400
-F 0 "#PWR017" H 7100 5150 50  0001 C CNN
+F 0 "#PWR6" H 7100 5150 50  0001 C CNN
 F 1 "GND" H 7100 5250 50  0000 C CNN
 F 2 "" H 7100 5400 60  0000 C CNN
@@
 NoConn ~ 7500 6750
 NoConn ~ 7500 6850
+$Comp
+L CONN_02X10 P1
+U 1 1 565A9401
+P 13450 9550
+F 0 "P1" H 13450 10100 50  0000 C CNN
+F 1 "CONN_02X10" V 13450 9550 50  0000 C CNN
+F 2 "Pin_Headers:Pin_Header_Straight_2x10" H 13450 8350 60  0000 C CNN
+F 3 "" H 13450 8350 60  0000 C CNN
+	1    13450 9550
+	1    0    0    -1
+$EndComp
+$Comp
+L CONN_02X10 P2
+U 1 1 565A97C1
+P 14350 9550
+F 0 "P2" H 14350 10100 50  0000 C CNN
+F 1 "CONN_02X10" V 14350 9550 50  0000 C CNN
+F 2 "Pin_Headers:Pin_Header_Straight_2x10" H 14350 8350 60  0000 C CNN
+F 3 "" H 14350 8350 60  0000 C CNN
+	1    14350 9550
+	1    0    0    -1
+$EndComp
 $EndSCHEMATC
