File: tinycom-a13/tinycom-a13.sch (KiCad schematic (older format))
At the start: 23 parts, among them P1 CONN_02X10, P2 CONN_02X10, U1 IC_A13, U2 H5TQ2G83BFR/FBGA82, Y1 Crystal

Commit message: a13 update
Parts:
- added P3: CONN_01X03, Pin_Headers:Pin_Header_Angled_1x03, symbol CONN_01X03
Connections:
- net labels added: UD0_N, UD0_P, UD1_N, UD1_P
- net labels removed: UDM0, UDM1, UDP0, UDP1
- wire segments 142 -> 144
Changed lines of the file:
@@
 LIBS:opendous
 LIBS:calculator
+LIBS:tinycom-a13-cache
 EELAYER 25 0
 EELAYER END
@@
 CSI_D7
 Text GLabel 7500 7350 0    60   Input ~ 0
-UDP1
+UD1_P
 Text GLabel 7500 7450 0    60   Input ~ 0
-UDM1
+UD1_N
 Text GLabel 7500 7550 0    60   Input ~ 0
-UDP0
+UD0_P
 Text GLabel 7500 7650 0    60   Input ~ 0
-UDM0
+UD0_N
 Text GLabel 7400 2200 0    60   Input ~ 0
 VCC_33
@@
 $EndComp
 $Comp
-L GND #PWR01
+L GND #PWR2
 U 1 1 5624C74D
 P 6400 5750
-F 0 "#PWR01" H 6400 5500 50  0001 C CNN
+F 0 "#PWR2" H 6400 5500 50  0001 C CNN
 F 1 "GND" H 6400 5600 50  0000 C CNN
 F 2 "" H 6400 5750 60  0000 C CNN
@@
 $EndComp
 $Comp
-L GND #PWR02
+L GND #PWR3
 U 1 1 5624C778
 P 6400 6050
-F 0 "#PWR02" H 6400 5800 50  0001 C CNN
+F 0 "#PWR3" H 6400 5800 50  0001 C CNN
 F 1 "GND" H 6400 5900 50  0000 C CNN
 F 2 "" H 6400 6050 60  0000 C CNN
@@
 VCC_14_CPU
 $Comp
-L +3.3V #PWR03
+L +3.3V #PWR8
 U 1 1 5624CB40
 P 7400 2200
-F 0 "#PWR03" H 7400 2050 50  0001 C CNN
+F 0 "#PWR8" H 7400 2050 50  0001 C CNN
 F 1 "+3.3V" H 7400 2340 50  0000 C CNN
 F 2 "" H 7400 2200 60  0000 C CNN
@@
 $EndComp
 $Comp
-L +1V5 #PWR04
+L +1V5 #PWR1
 U 1 1 5624CB62
 P 5250 2150
-F 0 "#PWR04" H 5250 2000 50  0001 C CNN
+F 0 "#PWR1" H 5250 2000 50  0001 C CNN
 F 1 "+1V5" H 5250 2290 50  0000 C CNN
 F 2 "" H 5250 2150 60  0000 C CNN
@@
 DDR3_BA2
 $Comp
-L +1V5 #PWR05
+L +1V5 #PWR17
 U 1 1 5625F72C
 P 15200 3600
-F 0 "#PWR05" H 15200 3450 50  0001 C CNN
+F 0 "#PWR17" H 15200 3450 50  0001 C CNN
 F 1 "+1V5" H 15200 3740 50  0000 C CNN
 F 2 "" H 15200 3600 60  0000 C CNN
@@
 $EndComp
 $Comp
-L GND #PWR06
+L GND #PWR18
 U 1 1 5625F96A
 P 15350 7200
-F 0 "#PWR06" H 15350 6950 50  0001 C CNN
+F 0 "#PWR18" H 15350 6950 50  0001 C CNN
 F 1 "GND" H 15350 7050 50  0000 C CNN
 F 2 "" H 15350 7200 60  0000 C CNN
@@
 DDR3_RST
 $Comp
-L GND #PWR07
+L GND #PWR10
 U 1 1 5625FBB8
 P 11800 5950
-F 0 "#PWR07" H 11800 5700 50  0001 C CNN
+F 0 "#PWR10" H 11800 5700 50  0001 C CNN
 F 1 "GND" H 11800 5800 50  0000 C CNN
 F 2 "" H 11800 5950 60  0000 C CNN
@@
 $EndComp
 $Comp
-L +1V5 #PWR08
+L +1V5 #PWR11
 U 1 1 5625FE07
 P 12000 7100
-F 0 "#PWR08" H 12000 6950 50  0001 C CNN
+F 0 "#PWR11" H 12000 6950 50  0001 C CNN
 F 1 "+1V5" H 12000 7240 50  0000 C CNN
 F 2 "" H 12000 7100 60  0000 C CNN
@@
 $EndComp
 $Comp
-L GND #PWR09
+L GND #PWR12
 U 1 1 5625FF1B
 P 12000 7850
-F 0 "#PWR09" H 12000 7600 50  0001 C CNN
+F 0 "#PWR12" H 12000 7600 50  0001 C CNN
 F 1 "GND" H 12000 7700 50  0000 C CNN
 F 2 "" H 12000 7850 60  0000 C CNN
@@
 $EndComp
 $Comp
-L GND #PWR010
+L GND #PWR13
 U 1 1 56260662
 P 12250 8100
-F 0 "#PWR010" H 12250 7850 50  0001 C CNN
+F 0 "#PWR13" H 12250 7850 50  0001 C CNN
 F 1 "GND" H 12250 7950 50  0000 C CNN
 F 2 "" H 12250 8100 60  0000 C CNN
@@
 NoConn ~ 15100 7350
 $Comp
-L GND #PWR011
+L GND #PWR14
 U 1 1 56261679
 P 12450 7900
-F 0 "#PWR011" H 12450 7650 50  0001 C CNN
+F 0 "#PWR14" H 12450 7650 50  0001 C CNN
 F 1 "GND" H 12450 7750 50  0000 C CNN
 F 2 "" H 12450 7900 60  0000 C CNN
@@
 $EndComp
 $Comp
-L GND #PWR012
+L GND #PWR9
 U 1 1 56262D84
 P 11100 7950
-F 0 "#PWR012" H 11100 7700 50  0001 C CNN
+F 0 "#PWR9" H 11100 7700 50  0001 C CNN
 F 1 "GND" H 11100 7800 50  0000 C CNN
 F 2 "" H 11100 7950 60  0000 C CNN
@@
 $EndComp
 $Comp
-L +1V5 #PWR013
+L +1V5 #PWR19
 U 1 1 562642D9
 P 16050 3500
-F 0 "#PWR013" H 16050 3350 50  0001 C CNN
+F 0 "#PWR19" H 16050 3350 50  0001 C CNN
 F 1 "+1V5" H 16050 3640 50  0000 C CNN
 F 2 "" H 16050 3500 60  0000 C CNN
@@
 $EndComp
 $Comp
-L GND #PWR014
+L GND #PWR20
 U 1 1 562643A7
 P 16100 3900
-F 0 "#PWR014" H 16100 3650 50  0001 C CNN
+F 0 "#PWR20" H 16100 3650 50  0001 C CNN
 F 1 "GND" H 16100 3750 50  0000 C CNN
 F 2 "" H 16100 3900 60  0000 C CNN
@@
 $EndComp
 $Comp
-L GND #PWR015
+L GND #PWR5
 U 1 1 56265943
 P 6850 3500
-F 0 "#PWR015" H 6850 3250 50  0001 C CNN
+F 0 "#PWR5" H 6850 3250 50  0001 C CNN
 F 1 "GND" H 6850 3350 50  0000 C CNN
 F 2 "" H 6850 3500 60  0000 C CNN
@@
 $EndComp
 $Comp
-L GND #PWR016
+L GND #PWR6
 U 1 1 56265988
 P 7050 2700
-F 0 "#PWR016" H 7050 2450 50  0001 C CNN
+F 0 "#PWR6" H 7050 2450 50  0001 C CNN
 F 1 "GND" H 7050 2550 50  0000 C CNN
 F 2 "" H 7050 2700 60  0000 C CNN
@@
 SVREF
 $Comp
-L GND #PWR017
+L GND #PWR7
 U 1 1 562A3A06
 P 7100 5400
-F 0 "#PWR017" H 7100 5150 50  0001 C CNN
+F 0 "#PWR7" H 7100 5150 50  0001 C CNN
 F 1 "GND" H 7100 5250 50  0000 C CNN
 F 2 "" H 7100 5400 60  0000 C CNN
@@
 $EndComp
 $Comp
-L GND #PWR018
+L GND #PWR15
 U 1 1 56ACB68E
 P 12800 9050
-F 0 "#PWR018" H 12800 8800 50  0001 C CNN
+F 0 "#PWR15" H 12800 8800 50  0001 C CNN
 F 1 "GND" H 12800 8900 50  0000 C CNN
 F 2 "" H 12800 9050 50  0000 C CNN
@@
 $EndComp
 $Comp
-L GND #PWR019
+L GND #PWR16
 U 1 1 56ACB7DE
 P 14600 9000
-F 0 "#PWR019" H 14600 8750 50  0001 C CNN
+F 0 "#PWR16" H 14600 8750 50  0001 C CNN
 F 1 "GND" H 14600 8850 50  0000 C CNN
 F 2 "" H 14600 9000 50  0000 C CNN
@@
 SDC0_D1
 Text GLabel 13000 9300 0    60   Input ~ 0
-UDP0
+UD0_P
 Text GLabel 13000 9400 0    60   Input ~ 0
-UDM0
+UD0_N
 Text GLabel 13000 9500 0    60   Input ~ 0
-UDP1
+UD1_P
 Text GLabel 13000 9600 0    60   Input ~ 0
-UDM1
-$Comp
-L GND #PWR?
+UD1_N
+$Comp
+L GND #PWR4
 U 1 1 56ACFC7E
 P 6600 4150
-F 0 "#PWR?" H 6600 3900 50  0001 C CNN
+F 0 "#PWR4" H 6600 3900 50  0001 C CNN
 F 1 "GND" H 6600 4000 50  0000 C CNN
 F 2 "" H 6600 4150 60  0000 C CNN
@@
 Wire Wire Line
 	6850 3200 6850 3050
+$Comp
+L CONN_01X03 P3
+U 1 1 56ACD7F3
+P 17550 9150
+F 0 "P3" H 17550 9350 50  0000 C CNN
+F 1 "CONN_01X03" V 17650 9150 50  0000 C CNN
+F 2 "Pin_Headers:Pin_Header_Angled_1x03" H 17550 9150 50  0000 C CNN
+F 3 "" H 17550 9150 50  0000 C CNN
+	1    17550 9150
+	1    0    0    -1
+$EndComp
+$Comp
+L GND #PWR21
+U 1 1 56ACD90E
+P 16550 9100
+F 0 "#PWR21" H 16550 8850 50  0001 C CNN
+F 1 "GND" H 16550 8950 50  0000 C CNN
+F 2 "" H 16550 9100 50  0000 C CNN
+F 3 "" H 16550 9100 50  0000 C CNN
+	1    16550 9100
+	1    0    0    -1
+$EndComp
+Wire Wire Line
+	16550 9050 17350 9050
+Text GLabel 17350 9150 0    60   Input ~ 0
+UART1_TX
+Wire Wire Line
+	16550 9050 16550 9100
+Text GLabel 17350 9250 0    60   Input ~ 0
+UART1_RX
 $EndSCHEMATC

Commit message: a12 update
Parts:
- added P4: CONN_01X01, symbol CONN_01X01
- added R5, R6: 240R, Resistors_SMD:R_0603, symbol R
Connections:
- net labels added: NMI_N, TWI0_SCK, TWI0_SDA
- wire segments 144 -> 150
- no-connect marks 76 -> 74

Commit message: fix a13 drc
Parts:
- R5, R6: value 240R -> 10K
Connections:
- net labels removed: CSI_CLK, CSI_D0, CSI_D1, CSI_D2, CSI_D3, CSI_D4, CSI_D5, CSI_D6, CSI_D7, CSI_HSYNC, CSI_MCLK, CSI_VSYNC, DDR3_D10, DDR3_D11, DDR3_D12, DDR3_D13, DDR3_D14, DDR3_D15, DDR3_D8, DDR3_D9, MICIN1
- no-connect marks 74 -> 95
Changed lines of the file:
@@
 Text GLabel 10900 5450 2    60   Input ~ 0
 DDR3_A14
-Text GLabel 10900 3150 2    60   Input ~ 0
-DDR3_D8
-Text GLabel 10900 3250 2    60   Input ~ 0
-DDR3_D9
-Text GLabel 10900 3350 2    60   Input ~ 0
-DDR3_D10
-Text GLabel 10900 3450 2    60   Input ~ 0
-DDR3_D11
-Text GLabel 10900 3550 2    60   Input ~ 0
-DDR3_D12
-Text GLabel 10900 3650 2    60   Input ~ 0
-DDR3_D13
-Text GLabel 10900 3750 2    60   Input ~ 0
-DDR3_D14
-Text GLabel 10900 3850 2    60   Input ~ 0
-DDR3_D15
 Text GLabel 10900 11450 2    60   Input ~ 0
 SDC0_D1
@@
 Text GLabel 10900 12550 2    60   Input ~ 0
 UART1_RX
-Text GLabel 10900 10150 2    60   Input ~ 0
-CSI_CLK
-Text GLabel 10900 10250 2    60   Input ~ 0
-CSI_MCLK
-Text GLabel 10900 10350 2    60   Input ~ 0
-CSI_HSYNC
-Text GLabel 10900 10450 2    60   Input ~ 0
-CSI_VSYNC
-Text GLabel 10900 10550 2    60   Input ~ 0
-CSI_D0
-Text GLabel 10900 10650 2    60   Input ~ 0
-CSI_D1
-Text GLabel 10900 10750 2    60   Input ~ 0
-CSI_D2
-Text GLabel 10900 10850 2    60   Input ~ 0
-CSI_D3
-Text GLabel 10900 10950 2    60   Input ~ 0
-CSI_D4
-Text GLabel 10900 11050 2    60   Input ~ 0
-CSI_D5
-Text GLabel 10900 11150 2    60   Input ~ 0
-CSI_D6
-Text GLabel 10900 11250 2    60   Input ~ 0
-CSI_D7
 Text GLabel 7500 7350 0    60   Input ~ 0
 UD1_P
@@
 	1    0    0    -1
 $EndComp
-Text GLabel 7500 8050 0    60   Input ~ 0
-MICIN1
 $Comp
 L H5TQ2G83BFR/FBGA82 U2
@@
 P 7200 6150
 F 0 "R5" V 7280 6150 50  0000 C CNN
-F 1 "240R" V 7200 6150 50  0000 C CNN
+F 1 "10K" V 7200 6150 50  0000 C CNN
 F 2 "Resistors_SMD:R_0603" V 7130 6150 30  0001 C CNN
 F 3 "" H 7200 6150 30  0000 C CNN
@@
 P 7200 6250
 F 0 "R6" V 7280 6250 50  0000 C CNN
-F 1 "240R" V 7200 6250 50  0000 C CNN
+F 1 "10K" V 7200 6250 50  0000 C CNN
 F 2 "Resistors_SMD:R_0603" V 7130 6250 30  0001 C CNN
 F 3 "" H 7200 6250 30  0000 C CNN
@@
 Wire Wire Line
 	15400 8950 15550 8950
+NoConn ~ 7500 8050
+NoConn ~ 10900 3150
+NoConn ~ 10900 3250
+NoConn ~ 10900 3350
+NoConn ~ 10900 3450
+NoConn ~ 10900 3550
+NoConn ~ 10900 3650
+NoConn ~ 10900 3750
+NoConn ~ 10900 3850
+NoConn ~ 10900 10150
+NoConn ~ 10900 10250
+NoConn ~ 10900 10350
+NoConn ~ 10900 10450
+NoConn ~ 10900 10550
+NoConn ~ 10900 10650
+NoConn ~ 10900 10750
+NoConn ~ 10900 10850
+NoConn ~ 10900 10950
+NoConn ~ 10900 11050
+NoConn ~ 10900 11150
+NoConn ~ 10900 11250
 $EndSCHEMATC

Commit message: a13 update
Parts:
- added C15: 100nF, Capacitors_SMD:C_0603, symbol C_Small
Connections:
- wire segments 150 -> 148
Other:
- moved on the sheet: C10, C7
Changed lines of the file:
@@
 L C_Small C10
 U 1 1 56267401
-P 6650 3300
-F 0 "C10" H 6660 3370 50  0000 L CNN
-F 1 "100nF" H 6660 3220 50  0000 L CNN
-F 2 "Capacitors_SMD:C_0603" H 6650 3300 60  0001 C CNN
-F 3 "" H 6650 3300 60  0000 C CNN
-	1    6650 3300
+P 6850 3300
+F 0 "C10" H 6860 3370 50  0000 L CNN
+F 1 "100nF" H 6860 3220 50  0000 L CNN
+F 2 "Capacitors_SMD:C_0603" H 6850 3300 60  0001 C CNN
+F 3 "" H 6850 3300 60  0000 C CNN
+	1    6850 3300
 	1    0    0    -1
 $EndComp
@@
 L C_Small C7
 U 1 1 562674C6
-P 6450 3300
-F 0 "C7" H 6460 3370 50  0000 L CNN
-F 1 "100nF" H 6460 3220 50  0000 L CNN
-F 2 "Capacitors_SMD:C_0603" H 6450 3300 60  0001 C CNN
-F 3 "" H 6450 3300 60  0000 C CNN
-	1    6450 3300
+P 7050 3300
+F 0 "C7" H 7060 3370 50  0000 L CNN
+F 1 "100nF" H 7060 3220 50  0000 L CNN
+F 2 "Capacitors_SMD:C_0603" H 7050 3300 60  0001 C CNN
+F 3 "" H 7050 3300 60  0000 C CNN
+	1    7050 3300
 	1    0    0    -1
 $EndComp
@@
 	7500 2550 7400 2550
 Connection ~ 7400 2550
-Wire Wire Line
-	7350 2450 7500 2450
 Connection ~ 7400 2450
 Wire Wire Line
@@
 Wire Wire Line
 	7400 3550 7500 3550
-Wire Wire Line
-	7500 3450 7400 3450
 Connection ~ 7400 3450
 Wire Wire Line
@@
 	7500 3150 7400 3150
 Connection ~ 7400 3150
-Wire Wire Line
-	6450 3050 7500 3050
 Connection ~ 7400 3050
 Wire Wire Line
@@
 Connection ~ 6900 2700
 Wire Wire Line
-	6450 3050 6450 3200
-Connection ~ 6850 3050
-Wire Wire Line
-	6650 3200 6650 3050
-Connection ~ 6650 3050
-Wire Wire Line
 	7050 3200 7050 3050
 Connection ~ 7050 3050
-Wire Wire Line
-	6450 3400 6450 3450
-Wire Wire Line
-	6450 3450 7050 3450
 Connection ~ 6850 3450
-Wire Wire Line
-	7050 3450 7050 3400
-Wire Wire Line
-	6650 3450 6650 3400
-Connection ~ 6650 3450
 Wire Wire Line
 	7350 6150 7500 6150
@@
 NoConn ~ 10900 11150
 NoConn ~ 10900 11250
+Wire Wire Line
+	7400 2450 7500 2450
+Wire Wire Line
+	6850 3050 7500 3050
+Wire Wire Line
+	7050 3400 7050 3450
+$Comp
+L C_Small C15
+U 1 1 56B0309F
+P 6500 5200
+F 0 "C15" H 6510 5270 50  0000 L CNN
+F 1 "100nF" H 6510 5120 50  0000 L CNN
+F 2 "Capacitors_SMD:C_0603" H 6500 5200 60  0001 C CNN
+F 3 "" H 6500 5200 60  0000 C CNN
+	1    6500 5200
+	1    0    0    -1
+$EndComp
+Wire Wire Line
+	6500 5050 6500 5100
+Connection ~ 6500 5050
+$Comp
+L GND #PWR022
+U 1 1 56B0330A
+P 6500 5400
+F 0 "#PWR022" H 6500 5150 50  0001 C CNN
+F 1 "GND" H 6500 5250 50  0000 C CNN
+F 2 "" H 6500 5400 60  0000 C CNN
+F 3 "" H 6500 5400 60  0000 C CNN
+	1    6500 5400
+	1    0    0    -1
+$EndComp
+Wire Wire Line
+	6500 5300 6500 5400
+Wire Wire Line
+	7050 3450 6850 3450
+Wire Wire Line
+	7500 3450 7400 3450
 $EndSCHEMATC

Commit message: a13 updte
Connections:
- net UD0_N: now also P1.6 (P6); no longer P1.10 (P10)
- net UD0_P: now also P1.4 (P4); no longer P1.8 (P8)
- net UD1_N: now also P1.10 (P10); no longer P1.14 (P14)
- net UD1_P: now also P1.8 (P8); no longer P1.12 (P12)
- net UART3_TX: now reaches U1.12 (PG9/SPI1_CS0/UART3_TX/EINT9)
- net UART3_TX: now also P2.4 (P4)
- net UART3_RX: now reaches U1.13 (PG10/SPI1_CLK/UART3_RX/EINT10)
- net UART3_RX: now also P2.6 (P6)
- no-connect marks 95 -> 93
Changed lines of the file:
@@
 NoConn ~ 10900 12250
 NoConn ~ 10900 12350
-NoConn ~ 10900 12650
-NoConn ~ 10900 12750
 NoConn ~ 10900 12850
 NoConn ~ 10900 12950
@@
 L GND #PWR018
 U 1 1 56ACB68E
-P 13650 9050
-F 0 "#PWR018" H 13650 8800 50  0001 C CNN
-F 1 "GND" H 13650 8900 50  0000 C CNN
-F 2 "" H 13650 9050 50  0000 C CNN
-F 3 "" H 13650 9050 50  0000 C CNN
-	1    13650 9050
+P 14000 9050
+F 0 "#PWR018" H 14000 8800 50  0001 C CNN
+F 1 "GND" H 14000 8900 50  0000 C CNN
+F 2 "" H 14000 9050 50  0000 C CNN
+F 3 "" H 14000 9050 50  0000 C CNN
+	1    14000 9050
 	1    0    0    -1
 $EndComp
@@
 L GND #PWR019
 U 1 1 56ACB7DE
-P 15550 8950
-F 0 "#PWR019" H 15550 8700 50  0001 C CNN
-F 1 "GND" H 15550 8800 50  0000 C CNN
-F 2 "" H 15550 8950 50  0000 C CNN
-F 3 "" H 15550 8950 50  0000 C CNN
-	1    15550 8950
+P 16000 8950
+F 0 "#PWR019" H 16000 8700 50  0001 C CNN
+F 1 "GND" H 16000 8800 50  0000 C CNN
+F 2 "" H 16000 8950 50  0000 C CNN
+F 3 "" H 16000 8950 50  0000 C CNN
+	1    16000 8950
 	1    0    0    -1
 $EndComp
@@
 Text GLabel 14900 9450 0    60   Input ~ 0
 SDC0_D1
+Text GLabel 13500 9100 2    60   Input ~ 0
+UD0_P
+Text GLabel 13500 9200 2    60   Input ~ 0
+UD0_N
 Text GLabel 13500 9300 2    60   Input ~ 0
-UD0_P
+UD1_P
 Text GLabel 13500 9400 2    60   Input ~ 0
-UD0_N
-Text GLabel 13500 9500 2    60   Input ~ 0
-UD1_P
-Text GLabel 13500 9600 2    60   Input ~ 0
 UD1_N
 $Comp
@@
 TWI0_SDA
 Wire Wire Line
-	13500 9000 13650 9000
-Wire Wire Line
-	13650 9000 13650 9050
-Wire Wire Line
-	15400 8950 15550 8950
+	13500 9000 14000 9000
+Wire Wire Line
+	15400 8950 16000 8950
 NoConn ~ 7500 8050
 NoConn ~ 10900 3150
@@
 Wire Wire Line
 	7500 3450 7400 3450
+Wire Wire Line
+	14000 9000 14000 9050
+Text GLabel 15400 9050 2    60   Input ~ 0
+UART3_TX
+Text GLabel 15400 9150 2    60   Input ~ 0
+UART3_RX
+Text GLabel 10900 12650 2    60   Input ~ 0
+UART3_TX
+Text GLabel 10900 12750 2    60   Input ~ 0
+UART3_RX
 $EndSCHEMATC
