File: tinycom-a13/tinycom-a13.kicad_pcb (KiCad board)
At the start: 4 copper layers, 39.4 x 40.7 mm, 23 parts, among them P1 CONN_02X10, P2 CONN_02X10, U1 IC_A13, U2 H5TQ2G83BFR/FBGA82, Y1 Crystal

Commit message: a13 update
Parts:
- added P3: CONN_01X03, Pin_Headers:Pin_Header_Angled_1x03, B.Cu at (87.4, 130.2)
- moved C7 2.67 mm to (108.5, 130.8)
- moved C12 0.63 mm to (112.0, 149.7)
- moved C13 0.62 mm to (114.5, 146.6)
Connections:
- net UDM0 renamed UD0_N
- net UDM1 renamed UD1_N
- net UDP0 renamed UD0_P
- net UDP1 renamed UD1_P
Routing:
- net VCC_14_INT: track 3.66 -> 96.8 mm, vias 2 -> 3
- net VCC_14_CPU: track 6.27 -> 56.2 mm
- net SDC0_D1: track 0.00 -> 35.9 mm, vias 0 -> 1
- net SDC0_D0: track 0.00 -> 33.1 mm, vias 0 -> 1
- net UART1_TX: track 0.00 -> 32.6 mm, vias 0 -> 1
- net UART1_RX: track 0.00 -> 30.3 mm, vias 0 -> 1
- net SDC0_CLK: track 0.00 -> 30.1 mm, vias 0 -> 1
- net SDC0_CMD: track 0.00 -> 27.4 mm, vias 0 -> 1
- net SDC0_D3: track 0.00 -> 25.9 mm, vias 0 -> 1
- net SDC0_D2: track 0.00 -> 24.2 mm, vias 0 -> 1
- net UD0_P: track 0.00 -> 17.1 mm, vias 0 -> 1
- net UD0_N: track 0.00 -> 16.3 mm, vias 0 -> 1
- net VCC_33: track 16.6 -> 30.8 mm
- net UD1_P: track 0.00 -> 12.7 mm, vias 0 -> 1
- net GND: track 26.3 -> 38.1 mm
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- added copper zone on In1.Cu, net GND
- added copper zone on In2.Cu, net VCC_15
- added copper zone on In2.Cu, net VCC_33
- removed copper zone on In2.Cu, net VCC_14
Other:
- net class Default: trace_width 0.15 -> 0.4

Commit message: a12 update
Parts:
- added R5: 240R, Resistors_SMD:R_0603, F.Cu at (120.4, 130.7)
- added R6: 240R, Resistors_SMD:R_0603, F.Cu at (121.8, 130.7)
- C3, C5: moved to F.Cu
- P1, P2: moved to B.Cu
- U1: footprint A13o:allwinner_a13-OLIMEX_IC_TQFP176 -> tinycom:allwinner_a13-OLIMEX_IC_TQFP176
- moved C3 17.0 mm to (86.5, 133.0), turned to 90 degrees
- moved C11 15.4 mm to (119.5, 139.7), turned to 270 degrees
- moved C12 13.9 mm to (112.9, 135.8), turned to 270 degrees
- moved C5 9.97 mm to (86.6, 150.4)
- moved C14 8.49 mm to (105.9, 133.4), turned to 270 degrees
- moved C4 7.60 mm to (102.3, 135.9), turned to 270 degrees
- moved C6 5.26 mm to (102.4, 142.6), turned to 90 degrees
- moved C9 2.81 mm to (109.5, 148.1), turned to 270 degrees
- moved P2 2.55 mm to (116.4, 123.8), turned to 90 degrees
- moved P1 2.54 mm to (93.9, 156.1), turned to 270 degrees
Connections:
- P1 pad 1: GND -> Net-(P1-Pad1)
- P1 pad 10: Net-(P1-Pad10) -> UD0_N
- P1 pad 11: UD1_P -> Net-(P1-Pad11)
- P1 pad 12: Net-(P1-Pad12) -> UD1_P
- P1 pad 13: UD1_N -> Net-(P1-Pad13)
- P1 pad 14: Net-(P1-Pad14) -> UD1_N
- P1 pad 2: Net-(P1-Pad2) -> GND
- P1 pad 7: UD0_P -> Net-(P1-Pad7)
- P1 pad 8: Net-(P1-Pad8) -> UD0_P
- P1 pad 9: UD0_N -> Net-(P1-Pad9)
- P2 pad 1: GND -> SDC0_D2
- P2 pad 10: SDC0_D0 -> VCC_30_ANL
- P2 pad 11: VCC_13_RTC -> SDC0_D1
- P2 pad 12: SDC0_D1 -> VCC_13_RTC
- P2 pad 13: VCC_15 -> Net-(P2-Pad13)
- P2 pad 14: Net-(P2-Pad14) -> VCC_15
- P2 pad 15: VCC_33 -> NMI_N
- P2 pad 16: Net-(P2-Pad16) -> VCC_33
- P2 pad 17: VCC_14_INT -> TWI0_SDA
- P2 pad 18: Net-(P2-Pad18) -> VCC_14_INT
- P2 pad 19: VCC_14_CPU -> TWI0_SCK
- P2 pad 2: SDC0_D2 -> GND
- P2 pad 20: Net-(P2-Pad20) -> VCC_14_CPU
- P2 pad 3: Net-(P2-Pad3) -> SDC0_D3
- P2 pad 4: SDC0_D3 -> Net-(P2-Pad4)
- P2 pad 5: Net-(P2-Pad5) -> SDC0_CMD
- P2 pad 6: SDC0_CMD -> Net-(P2-Pad6)
- P2 pad 7: Net-(P2-Pad7) -> SDC0_CLK
- P2 pad 8: SDC0_CLK -> Net-(P2-Pad8)
- P2 pad 9: VCC_30_ANL -> SDC0_D0
- U1 pad 101: Net-(U1-Pad101) -> TWI0_SCK
- U1 pad 102: Net-(U1-Pad102) -> TWI0_SDA
- U1 pad 157: VCC_33 -> Net-(P4-Pad1)
- U1 pad 158: VCC_33 -> NMI_N
- U1 pad 159: VCC_33 -> Net-(R5-Pad1)
Routing:
- net TWI0_SCK: track 0.00 -> 35.7 mm, vias 0 -> 2
- net SVREF: track 1.27 -> 36.4 mm, vias 0 -> 4
- net TWI0_SDA: track 0.00 -> 34.3 mm, vias 0 -> 2
- net VCC_30_ANL: track 0.00 -> 34.1 mm, vias 0 -> 2
- net NMI_N: track 0.00 -> 28.2 mm, vias 0 -> 1
- net VCC_15: track 18.2 -> 37.5 mm, vias 4 -> 22
- net VCC_14_INT: track 96.8 -> 113.9 mm, vias 3 -> 5
- net VCC_33: track 30.8 -> 25.6 mm, vias 4 -> 11
- net Net-(R5-Pad1): track 0.00 -> 5.08 mm
- net GND: track 38.1 -> 42.4 mm, vias 14 -> 29
- net UART1_TX: track 32.6 -> 33.9 mm
- net DDR3_A12: track 7.46 -> 6.87 mm
- net (no net): vias 11 -> 0
Other:
- net class Default: trace_width 0.4 -> 0.15

Commit message: fix a13 drc
Parts:
- R5, R6: value 240R -> 10K
- moved C8 1.04 mm to (105.2, 147.4), turned to 90 degrees
Connections:
- net CSI_CLK renamed Net-(U1-Pad114)
- net CSI_D0 renamed Net-(U1-Pad118)
- net CSI_D1 renamed Net-(U1-Pad119)
- net CSI_D2 renamed Net-(U1-Pad120)
- net CSI_D3 renamed Net-(U1-Pad121)
- net CSI_D4 renamed Net-(U1-Pad122)
- net CSI_D5 renamed Net-(U1-Pad123)
- net CSI_D6 renamed Net-(U1-Pad124)
- net CSI_D7 renamed Net-(U1-Pad125)
- net CSI_HSYNC renamed Net-(U1-Pad116)
- net CSI_MCLK renamed Net-(U1-Pad115)
- net CSI_VSYNC renamed Net-(U1-Pad117)
- net DDR3_D10 renamed Net-(U1-Pad39)
- net DDR3_D11 renamed Net-(U1-Pad24)
- net DDR3_D12 renamed Net-(U1-Pad36)
- net DDR3_D13 renamed Net-(U1-Pad26)
- net DDR3_D14 renamed Net-(U1-Pad38)
- net DDR3_D15 renamed Net-(U1-Pad27)
- net DDR3_D8 renamed Net-(U1-Pad37)
- net DDR3_D9 renamed Net-(U1-Pad25)
- net MICIN1 renamed Net-(U1-Pad84)

Commit message: a13 update
Parts:
- added C15: 100nF, Capacitors_SMD:C_0603, B.Cu at (107.8, 148.4)
Routing:
- net GND: vias 29 -> 30

Commit message: a13 updte
Connections:
- P1 pad 10: UD0_N -> UD1_N
- P1 pad 12: UD1_P -> Net-(P1-Pad12)
- P1 pad 14: UD1_N -> Net-(P1-Pad14)
- P1 pad 4: Net-(P1-Pad4) -> UD0_P
- P1 pad 6: Net-(P1-Pad6) -> UD0_N
- P1 pad 8: UD0_P -> UD1_P
- P2 pad 4: Net-(P2-Pad4) -> UART3_TX
- P2 pad 6: Net-(P2-Pad6) -> UART3_RX
- U1 pad 12: Net-(U1-Pad12) -> UART3_TX
- U1 pad 13: Net-(U1-Pad13) -> UART3_RX
Routing:
- net UART3_TX: track 0.00 -> 14.4 mm
- net UART3_RX: track 0.00 -> 12.8 mm
- net UD0_P: track 17.1 -> 23.0 mm
- net UD0_N: track 16.1 -> 21.2 mm
- net UD1_N: track 11.3 -> 15.9 mm
- net UD1_P: track 12.5 -> 17.0 mm
