File: tinycom-base/tinycom-base.sch (KiCad schematic (older format))
At the start: 28 parts, among them J1 MICRO_SD_HINGE, P1 CONN_02X10, P2 CONN_02X10, P3 USB_A, P4 USB_OTG, U1 SY8008BAAC, U2 SY8008BAAC, U3 SY8008BAAC, U4 RTL8188, U5 rainsun-antenna

Commit message: before resize vias
Parts:
- added P5: CONN_01X03, Pin_Headers:Pin_Header_Angled_1x03, symbol CONN_01X03
Connections:
- wire segments 117 -> 120
Changed lines of the file:
@@
 $EndComp
 $Comp
-L +5V #PWR01
+L +5V #PWR14
 U 1 1 562DA8F7
 P 5250 4200
-F 0 "#PWR01" H 5250 4050 50  0001 C CNN
+F 0 "#PWR14" H 5250 4050 50  0001 C CNN
 F 1 "+5V" H 5250 4340 50  0000 C CNN
 F 2 "" H 5250 4200 60  0000 C CNN
@@
 $EndComp
 $Comp
-L GND #PWR02
+L GND #PWR15
 U 1 1 562DA928
 P 5250 4600
-F 0 "#PWR02" H 5250 4350 50  0001 C CNN
+F 0 "#PWR15" H 5250 4350 50  0001 C CNN
 F 1 "GND" H 5250 4450 50  0000 C CNN
 F 2 "" H 5250 4600 60  0000 C CNN
@@
 UD0_P
 $Comp
-L +5V #PWR03
+L +5V #PWR16
 U 1 1 562DAC42
 P 5300 5050
-F 0 "#PWR03" H 5300 4900 50  0001 C CNN
+F 0 "#PWR16" H 5300 4900 50  0001 C CNN
 F 1 "+5V" H 5300 5190 50  0000 C CNN
 F 2 "" H 5300 5050 60  0000 C CNN
@@
 $EndComp
 $Comp
-L GND #PWR04
+L GND #PWR17
 U 1 1 562DAC77
 P 5300 5500
-F 0 "#PWR04" H 5300 5250 50  0001 C CNN
+F 0 "#PWR17" H 5300 5250 50  0001 C CNN
 F 1 "GND" H 5300 5350 50  0000 C CNN
 F 2 "" H 5300 5500 60  0000 C CNN
@@
 UD1_P
 $Comp
-L GND #PWR05
+L GND #PWR5
 U 1 1 562DAF0B
 P 1350 1750
-F 0 "#PWR05" H 1350 1500 50  0001 C CNN
+F 0 "#PWR5" H 1350 1500 50  0001 C CNN
 F 1 "GND" H 1350 1600 50  0000 C CNN
 F 2 "" H 1350 1750 60  0000 C CNN
@@
 $EndComp
 $Comp
-L +5V #PWR06
+L +5V #PWR3
 U 1 1 562DAF87
 P 1250 1350
-F 0 "#PWR06" H 1250 1200 50  0001 C CNN
+F 0 "#PWR3" H 1250 1200 50  0001 C CNN
 F 1 "+5V" H 1250 1490 50  0000 C CNN
 F 2 "" H 1250 1350 60  0000 C CNN
@@
 $EndComp
 $Comp
-L +5V #PWR07
+L +5V #PWR1
 U 1 1 562DB0A5
 P 1150 2550
-F 0 "#PWR07" H 1150 2400 50  0001 C CNN
+F 0 "#PWR1" H 1150 2400 50  0001 C CNN
 F 1 "+5V" H 1150 2690 50  0000 C CNN
 F 2 "" H 1150 2550 60  0000 C CNN
@@
 $EndComp
 $Comp
-L GND #PWR08
+L GND #PWR6
 U 1 1 562DB1B7
 P 1350 2900
-F 0 "#PWR08" H 1350 2650 50  0001 C CNN
+F 0 "#PWR6" H 1350 2650 50  0001 C CNN
 F 1 "GND" H 1350 2750 50  0000 C CNN
 F 2 "" H 1350 2900 60  0000 C CNN
@@
 $EndComp
 $Comp
-L +5V #PWR09
+L +5V #PWR2
 U 1 1 562DB2B7
 P 1150 3800
-F 0 "#PWR09" H 1150 3650 50  0001 C CNN
+F 0 "#PWR2" H 1150 3650 50  0001 C CNN
 F 1 "+5V" H 1150 3940 50  0000 C CNN
 F 2 "" H 1150 3800 60  0000 C CNN
@@
 $EndComp
 $Comp
-L GND #PWR010
+L GND #PWR4
 U 1 1 562DB346
 P 1300 4150
-F 0 "#PWR010" H 1300 3900 50  0001 C CNN
+F 0 "#PWR4" H 1300 3900 50  0001 C CNN
 F 1 "GND" H 1300 4000 50  0000 C CNN
 F 2 "" H 1300 4150 60  0000 C CNN
@@
 UD1_P
 $Comp
-L GND #PWR011
+L GND #PWR18
 U 1 1 562DAEC4
 P 5800 6000
-F 0 "#PWR011" H 5800 5750 50  0001 C CNN
+F 0 "#PWR18" H 5800 5750 50  0001 C CNN
 F 1 "GND" H 5800 5850 50  0000 C CNN
 F 2 "" H 5800 6000 60  0000 C CNN
@@
 $EndComp
 $Comp
-L GND #PWR012
+L GND #PWR19
 U 1 1 562DA997
 P 6400 7200
-F 0 "#PWR012" H 6400 6950 50  0001 C CNN
+F 0 "#PWR19" H 6400 6950 50  0001 C CNN
 F 1 "GND" H 6400 7050 50  0000 C CNN
 F 2 "" H 6400 7200 60  0000 C CNN
@@
 SDC0_D1
 $Comp
-L GND #PWR013
+L GND #PWR22
 U 1 1 562DAEE9
 P 7450 4950
-F 0 "#PWR013" H 7450 4700 50  0001 C CNN
+F 0 "#PWR22" H 7450 4700 50  0001 C CNN
 F 1 "GND" H 7450 4800 50  0000 C CNN
 F 2 "" H 7450 4950 60  0000 C CNN
@@
 $EndComp
 $Comp
-L GND #PWR014
+L GND #PWR24
 U 1 1 562DAF47
 P 9050 5450
-F 0 "#PWR014" H 9050 5200 50  0001 C CNN
+F 0 "#PWR24" H 9050 5200 50  0001 C CNN
 F 1 "GND" H 9050 5300 50  0000 C CNN
 F 2 "" H 9050 5450 60  0000 C CNN
@@
 $EndComp
 $Comp
-L +3.3V #PWR015
+L +3.3V #PWR21
 U 1 1 562DB369
 P 7300 4000
-F 0 "#PWR015" H 7300 3850 50  0001 C CNN
+F 0 "#PWR21" H 7300 3850 50  0001 C CNN
 F 1 "+3.3V" H 7300 4140 50  0000 C CNN
 F 2 "" H 7300 4000 60  0000 C CNN
@@
 $EndComp
 $Comp
-L GND #PWR016
+L GND #PWR9
 U 1 1 562DB89F
 P 3250 2000
-F 0 "#PWR016" H 3250 1750 50  0001 C CNN
+F 0 "#PWR9" H 3250 1750 50  0001 C CNN
 F 1 "GND" H 3250 1850 50  0000 C CNN
 F 2 "" H 3250 2000 60  0000 C CNN
@@
 $EndComp
 $Comp
-L +3.3V #PWR017
+L +3.3V #PWR10
 U 1 1 562DBC47
 P 3600 1350
-F 0 "#PWR017" H 3600 1200 50  0001 C CNN
+F 0 "#PWR10" H 3600 1200 50  0001 C CNN
 F 1 "+3.3V" H 3600 1490 50  0000 C CNN
 F 2 "" H 3600 1350 60  0000 C CNN
@@
 $EndComp
 $Comp
-L GND #PWR018
+L GND #PWR8
 U 1 1 562F8BF0
 P 3150 3150
-F 0 "#PWR018" H 3150 2900 50  0001 C CNN
+F 0 "#PWR8" H 3150 2900 50  0001 C CNN
 F 1 "GND" H 3150 3000 50  0000 C CNN
 F 2 "" H 3150 3150 60  0000 C CNN
@@
 $EndComp
 $Comp
-L GND #PWR019
+L GND #PWR7
 U 1 1 562F9FD4
 P 3100 4550
-F 0 "#PWR019" H 3100 4300 50  0001 C CNN
+F 0 "#PWR7" H 3100 4300 50  0001 C CNN
 F 1 "GND" H 3100 4400 50  0000 C CNN
 F 2 "" H 3100 4550 60  0000 C CNN
@@
 $EndComp
 $Comp
-L GND #PWR020
+L GND #PWR11
 U 1 1 56336272
 P 4400 1900
-F 0 "#PWR020" H 4400 1650 50  0001 C CNN
+F 0 "#PWR11" H 4400 1650 50  0001 C CNN
 F 1 "GND" H 4400 1750 50  0000 C CNN
 F 2 "" H 4400 1900 60  0000 C CNN
@@
 $EndComp
 $Comp
-L GND #PWR021
+L GND #PWR12
 U 1 1 5634B03F
 P 4900 4550
-F 0 "#PWR021" H 4900 4300 50  0001 C CNN
+F 0 "#PWR12" H 4900 4300 50  0001 C CNN
 F 1 "GND" H 4900 4400 50  0000 C CNN
 F 2 "" H 4900 4550 60  0000 C CNN
@@
 $EndComp
 $Comp
-L GND #PWR022
+L GND #PWR13
 U 1 1 5634B0B0
 P 4900 5400
-F 0 "#PWR022" H 4900 5150 50  0001 C CNN
+F 0 "#PWR13" H 4900 5150 50  0001 C CNN
 F 1 "GND" H 4900 5250 50  0000 C CNN
 F 2 "" H 4900 5400 60  0000 C CNN
@@
 $EndComp
 $Comp
-L GND #PWR023
+L GND #PWR23
 U 1 1 565A1BF7
 P 8250 6000
-F 0 "#PWR023" H 8250 5750 50  0001 C CNN
+F 0 "#PWR23" H 8250 5750 50  0001 C CNN
 F 1 "GND" H 8250 5850 50  0000 C CNN
 F 2 "" H 8250 6000 60  0000 C CNN
@@
 	8250 5950 8250 6000
 $Comp
-L GND #PWR024
+L GND #PWR20
 U 1 1 565A1DA6
 P 7100 5650
-F 0 "#PWR024" H 7100 5400 50  0001 C CNN
+F 0 "#PWR20" H 7100 5400 50  0001 C CNN
 F 1 "GND" H 7100 5500 50  0000 C CNN
 F 2 "" H 7100 5650 60  0000 C CNN
@@
 	8650 5850 8650 5900
 $Comp
-L GND #PWR025
+L GND #PWR25
 U 1 1 565A4582
 P 9250 6000
-F 0 "#PWR025" H 9250 5750 50  0001 C CNN
+F 0 "#PWR25" H 9250 5750 50  0001 C CNN
 F 1 "GND" H 9250 5850 50  0000 C CNN
 F 2 "" H 9250 6000 60  0000 C CNN
@@
 HPCOM
 Text GLabel 6500 7050 0    60   Input ~ 0
+UART0_TX
+Text GLabel 6500 6950 0    60   Input ~ 0
 UART0_RX
-Text GLabel 6500 6950 0    60   Input ~ 0
-UART0_TX
 Text GLabel 7000 6250 2    60   Input ~ 0
 SATA_TXP
@@
 Wire Wire Line
 	1150 2650 1400 2650
+$Comp
+L CONN_01X03 P5
+U 1 1 56629594
+P 2950 6500
+F 0 "P5" H 2950 6700 50  0000 C CNN
+F 1 "CONN_01X03" V 3050 6500 50  0000 C CNN
+F 2 "Pin_Headers:Pin_Header_Angled_1x03" H 2950 6500 50  0000 C CNN
+F 3 "" H 2950 6500 50  0000 C CNN
+	1    2950 6500
+	1    0    0    -1
+$EndComp
+$Comp
+L GND #PWR?
+U 1 1 56629D5C
+P 2600 6300
+F 0 "#PWR?" H 2600 6050 50  0001 C CNN
+F 1 "GND" H 2600 6150 50  0000 C CNN
+F 2 "" H 2600 6300 50  0000 C CNN
+F 3 "" H 2600 6300 50  0000 C CNN
+	1    2600 6300
+	1    0    0    -1
+$EndComp
+Wire Wire Line
+	2750 6400 2750 6250
+Wire Wire Line
+	2750 6250 2600 6250
+Wire Wire Line
+	2600 6250 2600 6300
+Text GLabel 2750 6500 0    60   Input ~ 0
+UART0_TX
+Text GLabel 2750 6600 0    60   Input ~ 0
+UART0_RX
 $EndSCHEMATC

Commit message: send production
Connections:
- wire segments 120 -> 121
Changed lines of the file:
@@
 $EndComp
 Text GLabel 5650 6850 2    60   Input ~ 0
+UD2_P
+Text GLabel 5650 6750 2    60   Input ~ 0
 UD2_N
-Text GLabel 5650 6750 2    60   Input ~ 0
-UD2_P
 Text GLabel 5650 6650 2    60   Input ~ 0
+UD1_P
+Text GLabel 5650 6550 2    60   Input ~ 0
 UD1_N
-Text GLabel 5650 6550 2    60   Input ~ 0
-UD1_P
 $Comp
 L GND #PWR18
@@
 	1    0    0    -1
 $EndComp
-$Comp
-L GND #PWR23
-U 1 1 565A1BF7
-P 8250 6000
-F 0 "#PWR23" H 8250 5750 50  0001 C CNN
-F 1 "GND" H 8250 5850 50  0000 C CNN
-F 2 "" H 8250 6000 60  0000 C CNN
-F 3 "" H 8250 6000 60  0000 C CNN
-	1    8250 6000
-	1    0    0    -1
-$EndComp
-Wire Wire Line
-	8150 5950 8250 5950
-Wire Wire Line
-	8250 5950 8250 6000
+Wire Wire Line
+	8150 5950 8650 5950
 $Comp
 L GND #PWR20
@@
 SDC0_D1
 Text GLabel 5650 6350 2    60   Input ~ 0
+UD0_N
+Text GLabel 5650 6450 2    60   Input ~ 0
 UD0_P
-Text GLabel 5650 6450 2    60   Input ~ 0
-UD0_N
 Wire Wire Line
 	8150 5850 8650 5850
 Wire Wire Line
 	8650 5850 8650 5900
-$Comp
-L GND #PWR25
-U 1 1 565A4582
-P 9250 6000
-F 0 "#PWR25" H 9250 5750 50  0001 C CNN
-F 1 "GND" H 9250 5850 50  0000 C CNN
-F 2 "" H 9250 6000 60  0000 C CNN
-F 3 "" H 9250 6000 60  0000 C CNN
-	1    9250 6000
-	1    0    0    -1
-$EndComp
 Wire Wire Line
 	9250 5900 9250 6000
@@
 Text GLabel 2750 6600 0    60   Input ~ 0
 UART0_RX
+Wire Wire Line
+	8650 5950 8650 6000
+Wire Wire Line
+	8650 6000 9250 6000
 $EndSCHEMATC

Commit message: a64 start ddr route
Parts:
- C11, C12: footprint Capacitors_Elko_ThroughHole:Elko_vert_11.2x6.3mm_RM2.5_CopperClear -> Capacitors_Tantalum_SMD:TantalC_SizeA_EIA-3216_Reflow
- C2, C5, C6, C7: footprint Capacitors_SMD:C_0805 -> Capacitors_SMD:C_1206
Changed lines of the file:
@@
 $EndComp
 $Comp
-L +5V #PWR14
+L +5V #PWR01
 U 1 1 562DA8F7
 P 5250 4200
-F 0 "#PWR14" H 5250 4050 50  0001 C CNN
+F 0 "#PWR01" H 5250 4050 50  0001 C CNN
 F 1 "+5V" H 5250 4340 50  0000 C CNN
 F 2 "" H 5250 4200 60  0000 C CNN
@@
 $EndComp
 $Comp
-L GND #PWR15
+L GND #PWR02
 U 1 1 562DA928
 P 5250 4600
-F 0 "#PWR15" H 5250 4350 50  0001 C CNN
+F 0 "#PWR02" H 5250 4350 50  0001 C CNN
 F 1 "GND" H 5250 4450 50  0000 C CNN
 F 2 "" H 5250 4600 60  0000 C CNN
@@
 UD0_P
 $Comp
-L +5V #PWR16
+L +5V #PWR03
 U 1 1 562DAC42
 P 5300 5050
-F 0 "#PWR16" H 5300 4900 50  0001 C CNN
+F 0 "#PWR03" H 5300 4900 50  0001 C CNN
 F 1 "+5V" H 5300 5190 50  0000 C CNN
 F 2 "" H 5300 5050 60  0000 C CNN
@@
 $EndComp
 $Comp
-L GND #PWR17
+L GND #PWR04
 U 1 1 562DAC77
 P 5300 5500
-F 0 "#PWR17" H 5300 5250 50  0001 C CNN
+F 0 "#PWR04" H 5300 5250 50  0001 C CNN
 F 1 "GND" H 5300 5350 50  0000 C CNN
 F 2 "" H 5300 5500 60  0000 C CNN
@@
 UD1_P
 $Comp
-L GND #PWR5
+L GND #PWR05
 U 1 1 562DAF0B
 P 1350 1750
-F 0 "#PWR5" H 1350 1500 50  0001 C CNN
+F 0 "#PWR05" H 1350 1500 50  0001 C CNN
 F 1 "GND" H 1350 1600 50  0000 C CNN
 F 2 "" H 1350 1750 60  0000 C CNN
@@
 $EndComp
 $Comp
-L +5V #PWR3
+L +5V #PWR06
 U 1 1 562DAF87
 P 1250 1350
-F 0 "#PWR3" H 1250 1200 50  0001 C CNN
+F 0 "#PWR06" H 1250 1200 50  0001 C CNN
 F 1 "+5V" H 1250 1490 50  0000 C CNN
 F 2 "" H 1250 1350 60  0000 C CNN
@@
 $EndComp
 $Comp
-L +5V #PWR1
+L +5V #PWR07
 U 1 1 562DB0A5
 P 1150 2550
-F 0 "#PWR1" H 1150 2400 50  0001 C CNN
+F 0 "#PWR07" H 1150 2400 50  0001 C CNN
 F 1 "+5V" H 1150 2690 50  0000 C CNN
 F 2 "" H 1150 2550 60  0000 C CNN
@@
 $EndComp
 $Comp
-L GND #PWR6
+L GND #PWR08
 U 1 1 562DB1B7
 P 1350 2900
-F 0 "#PWR6" H 1350 2650 50  0001 C CNN
+F 0 "#PWR08" H 1350 2650 50  0001 C CNN
 F 1 "GND" H 1350 2750 50  0000 C CNN
 F 2 "" H 1350 2900 60  0000 C CNN
@@
 $EndComp
 $Comp
-L +5V #PWR2
+L +5V #PWR09
 U 1 1 562DB2B7
 P 1150 3800
-F 0 "#PWR2" H 1150 3650 50  0001 C CNN
+F 0 "#PWR09" H 1150 3650 50  0001 C CNN
 F 1 "+5V" H 1150 3940 50  0000 C CNN
 F 2 "" H 1150 3800 60  0000 C CNN
@@
 $EndComp
 $Comp
-L GND #PWR4
+L GND #PWR010
 U 1 1 562DB346
 P 1300 4150
-F 0 "#PWR4" H 1300 3900 50  0001 C CNN
+F 0 "#PWR010" H 1300 3900 50  0001 C CNN
 F 1 "GND" H 1300 4000 50  0000 C CNN
 F 2 "" H 1300 4150 60  0000 C CNN
@@
 UD1_N
 $Comp
-L GND #PWR18
+L GND #PWR011
 U 1 1 562DAEC4
 P 5800 6000
-F 0 "#PWR18" H 5800 5750 50  0001 C CNN
+F 0 "#PWR011" H 5800 5750 50  0001 C CNN
 F 1 "GND" H 5800 5850 50  0000 C CNN
 F 2 "" H 5800 6000 60  0000 C CNN
@@
 $EndComp
 $Comp
-L GND #PWR19
+L GND #PWR012
 U 1 1 562DA997
 P 6400 7200
-F 0 "#PWR19" H 6400 6950 50  0001 C CNN
+F 0 "#PWR012" H 6400 6950 50  0001 C CNN
 F 1 "GND" H 6400 7050 50  0000 C CNN
 F 2 "" H 6400 7200 60  0000 C CNN
@@
 SDC0_D1
 $Comp
-L GND #PWR22
+L GND #PWR013
 U 1 1 562DAEE9
 P 7450 4950
-F 0 "#PWR22" H 7450 4700 50  0001 C CNN
+F 0 "#PWR013" H 7450 4700 50  0001 C CNN
 F 1 "GND" H 7450 4800 50  0000 C CNN
 F 2 "" H 7450 4950 60  0000 C CNN
@@
 $EndComp
 $Comp
-L GND #PWR24
+L GND #PWR014
 U 1 1 562DAF47
 P 9050 5450
-F 0 "#PWR24" H 9050 5200 50  0001 C CNN
+F 0 "#PWR014" H 9050 5200 50  0001 C CNN
 F 1 "GND" H 9050 5300 50  0000 C CNN
 F 2 "" H 9050 5450 60  0000 C CNN
@@
 $EndComp
 $Comp
-L +3.3V #PWR21
+L +3.3V #PWR015
 U 1 1 562DB369
 P 7300 4000
-F 0 "#PWR21" H 7300 3850 50  0001 C CNN
+F 0 "#PWR015" H 7300 3850 50  0001 C CNN
 F 1 "+3.3V" H 7300 4140 50  0000 C CNN
 F 2 "" H 7300 4000 60  0000 C CNN
@@
 $EndComp
 $Comp
-L GND #PWR9
+L GND #PWR016
 U 1 1 562DB89F
 P 3250 2000
-F 0 "#PWR9" H 3250 1750 50  0001 C CNN
+F 0 "#PWR016" H 3250 1750 50  0001 C CNN
 F 1 "GND" H 3250 1850 50  0000 C CNN
 F 2 "" H 3250 2000 60  0000 C CNN
@@
 $EndComp
 $Comp
-L +3.3V #PWR10
+L +3.3V #PWR017
 U 1 1 562DBC47
 P 3600 1350
-F 0 "#PWR10" H 3600 1200 50  0001 C CNN
+F 0 "#PWR017" H 3600 1200 50  0001 C CNN
 F 1 "+3.3V" H 3600 1490 50  0000 C CNN
 F 2 "" H 3600 1350 60  0000 C CNN
@@
 F 0 "C2" H 3710 1720 50  0000 L CNN
 F 1 "C_Small" H 3710 1570 50  0000 L CNN
-F 2 "Capacitors_SMD:C_0805" H 3700 1650 60  0001 C CNN
+F 2 "Capacitors_SMD:C_1206" H 3700 1650 60  0001 C CNN
 F 3 "" H 3700 1650 60  0000 C CNN
 	1    3700 1650
@@
 F 0 "C6" H 3560 2970 50  0000 L CNN
 F 1 "C_Small" H 3560 2820 50  0000 L CNN
-F 2 "Capacitors_SMD:C_0805" H 3550 2900 60  0001 C CNN
+F 2 "Capacitors_SMD:C_1206" H 3550 2900 60  0001 C CNN
 F 3 "" H 3550 2900 60  0000 C CNN
 	1    3550 2900
@@
 $EndComp
 $Comp
-L GND #PWR8
+L GND #PWR018
 U 1 1 562F8BF0
 P 3150 3150
-F 0 "#PWR8" H 3150 2900 50  0001 C CNN
+F 0 "#PWR018" H 3150 2900 50  0001 C CNN
 F 1 "GND" H 3150 3000 50  0000 C CNN
 F 2 "" H 3150 3150 60  0000 C CNN
@@
 F 0 "C5" H 3460 4220 50  0000 L CNN
 F 1 "C_Small" H 3460 4070 50  0000 L CNN
-F 2 "Capacitors_SMD:C_0805" H 3450 4150 60  0001 C CNN
+F 2 "Capacitors_SMD:C_1206" H 3450 4150 60  0001 C CNN
 F 3 "" H 3450 4150 60  0000 C CNN
 	1    3450 4150
@@
 $EndComp
 $Comp
-L GND #PWR7
+L GND #PWR019
 U 1 1 562F9FD4
 P 3100 4550
-F 0 "#PWR7" H 3100 4300 50  0001 C CNN
+F 0 "#PWR019" H 3100 4300 50  0001 C CNN
 F 1 "GND" H 3100 4400 50  0000 C CNN
 F 2 "" H 3100 4550 60  0000 C CNN
@@
 $EndComp
 $Comp
-L GND #PWR11
+L GND #PWR020
 U 1 1 56336272
 P 4400 1900
-F 0 "#PWR11" H 4400 1650 50  0001 C CNN
+F 0 "#PWR020" H 4400 1650 50  0001 C CNN
 F 1 "GND" H 4400 1750 50  0000 C CNN
 F 2 "" H 4400 1900 60  0000 C CNN
@@
 F 0 "C7" H 4760 1720 50  0000 L CNN
 F 1 "C_Small" H 4760 1570 50  0000 L CNN
-F 2 "Capacitors_SMD:C_0805" H 4750 1650 60  0001 C CNN
+F 2 "Capacitors_SMD:C_1206" H 4750 1650 60  0001 C CNN
 F 3 "" H 4750 1650 60  0000 C CNN
 	1    4750 1650
@@
 $EndComp
 $Comp
-L GND #PWR12
+L GND #PWR021
 U 1 1 5634B03F
 P 4900 4550
-F 0 "#PWR12" H 4900 4300 50  0001 C CNN
+F 0 "#PWR021" H 4900 4300 50  0001 C CNN
 F 1 "GND" H 4900 4400 50  0000 C CNN
 F 2 "" H 4900 4550 60  0000 C CNN
@@
 $EndComp
 $Comp
-L GND #PWR13
+L GND #PWR022
 U 1 1 5634B0B0
 P 4900 5400
-F 0 "#PWR13" H 4900 5150 50  0001 C CNN
+F 0 "#PWR022" H 4900 5150 50  0001 C CNN
 F 1 "GND" H 4900 5250 50  0000 C CNN
 F 2 "" H 4900 5400 60  0000 C CNN
@@
 F 0 "C11" H 4610 5320 50  0000 L CNN
 F 1 "CP_Small" H 4610 5170 50  0000 L CNN
-F 2 "Capacitors_Elko_ThroughHole:Elko_vert_11.2x6.3mm_RM2.5_CopperClear" H 4600 5250 60  0001 C CNN
+F 2 "Capacitors_Tantalum_SMD:TantalC_SizeA_EIA-3216_Reflow" H 4600 5250 60  0001 C CNN
 F 3 "" H 4600 5250 60  0000 C CNN
 	1    4600 5250
@@
 F 0 "C12" H 4660 4470 50  0000 L CNN
 F 1 "CP_Small" H 4660 4320 50  0000 L CNN
-F 2 "Capacitors_Elko_ThroughHole:Elko_vert_11.2x6.3mm_RM2.5_CopperClear" H 4650 4400 60  0001 C CNN
+F 2 "Capacitors_Tantalum_SMD:TantalC_SizeA_EIA-3216_Reflow" H 4650 4400 60  0001 C CNN
 F 3 "" H 4650 4400 60  0000 C CNN
 	1    4650 4400
@@
 	8150 5950 8650 5950
 $Comp
-L GND #PWR20
+L GND #PWR023
 U 1 1 565A1DA6
 P 7100 5650
-F 0 "#PWR20" H 7100 5400 50  0001 C CNN
+F 0 "#PWR023" H 7100 5400 50  0001 C CNN
 F 1 "GND" H 7100 5500 50  0000 C CNN
 F 2 "" H 7100 5650 60  0000 C CNN
@@
 $EndComp
 $Comp
-L GND #PWR?
+L GND #PWR024
 U 1 1 56629D5C
 P 2600 6300
-F 0 "#PWR?" H 2600 6050 50  0001 C CNN
+F 0 "#PWR024" H 2600 6050 50  0001 C CNN
 F 1 "GND" H 2600 6150 50  0000 C CNN
 F 2 "" H 2600 6300 50  0000 C CNN

Commit message: reroute, escape bga
Parts:
- removed D1: D_Schottky_Small, Diodes_SMD:SMA_Standard, symbol D_Schottky_Small
- removed P5: CONN_01X03, Pin_Headers:Pin_Header_Angled_1x03, symbol CONN_01X03
- removed R7: R_Small, Resistors_SMD:R_0805, symbol R_Small
- removed U2: SY8008BAAC, opendous:SOT23-5_Opendous, symbol SY8008BAAC
- added C1, C3: C_Small, Capacitors_SMD:C_1206, symbol C_Small
- added C10, C4, C9: C_Small, Capacitors_SMD:C_0805, symbol C_Small
- added L4: SMD-INDUCTOR-2.2UH-20%-1.2A(0805), cd32:CD32, symbol SMD-INDUCTOR-2.2UH-20%-1.2A(0805)
- added U2: OLIMEX_IC_AXP209, ax209:ax209-OLIMEX_IC_QFN48, symbol OLIMEX_IC_AXP209
- C6, C7: footprint Capacitors_SMD:C_1206 -> Capacitors_SMD:C_0805
- R5: value R_Small -> 2.2K
- R6: value R_Small -> 200K
Connections:
- net labels added: IPSOUT, NMI_N, TWI0_SCK, TWI0_SDA, UART1_RX, UART1_TX, VCC_12_CPU, VCC_12_INT, VCC_30_ANL, VCC_30_RTC
- net labels removed: HPCOM, HPL, HPR, SATA_RXM, SATA_RXP, SATA_TXM, SATA_TXP, UART0_RX, UART0_TX, VCC_12, VCC_30
- wire segments 121 -> 132
- no-connect marks 0 -> 23
Other:
- moved on the sheet: C2, C5, L1, L3, P1, P2, R1, R2, R3, R4, U1, U3

Commit message: routing
Parts:
- added C13, C14: 10uF, Capacitors_SMD:C_0805, symbol C_Small
- added R7, R8: 2.2K, Resistors_SMD:R_0805, symbol R_Small
- U2: value OLIMEX_IC_AXP209 -> AXP209; footprint ax209:ax209-OLIMEX_IC_QFN48 -> tinycom:ax209; symbol OLIMEX_IC_AXP209 -> OLIMEX_IC_AXP209-RESCUE-tinycom-base
Connections:
- net UD2_N is gone; now on net UD1_N: U4.3
- net UD2_P is gone; now on net UD1_P: U4.2
- net +3V3: now also R7.2, R8.2
- net GND: now also C13.1, C14.1
- net IPSOUT: now also C13.2, C14.2
- net TWI0_SCK: now also R8.1
- net TWI0_SDA: now also R7.1
- net UD0_N: now also P3.2 (D-)
- net UD0_P: now also P3.3 (D+)
- net UD1_N: no longer P3.2 (D-)
- net UD1_P: no longer P3.3 (D+)

Commit message: pics
Parts:
- U2: symbol OLIMEX_IC_AXP209-RESCUE-tinycom-base -> OLIMEX_IC_AXP209-RESCUE-tinycom-base-RESCUE-tinycom-base
Connections:
- net GND: now also U2.N1 (GND_PAD); no longer U2.~ (GND_PAD)
Changed lines of the file:
@@
 UART1_TX
 $Comp
-L OLIMEX_IC_AXP209-RESCUE-tinycom-base U2
+L OLIMEX_IC_AXP209-RESCUE-tinycom-base-RESCUE-tinycom-base U2
 U 1 1 567CCBE4
 P 2200 3350
