File: tinycom-a64/tinycom-a64.sch (KiCad schematic (older format))
At the start: 28 parts, among them P1 CONN_02X10, P2 CONN_02X10, U1 AllWinner-A64(FBGA396), U2 H5TQG63BFR/FBGA96, Y1 Crystal

Commit message: a64 update
Parts:
- added P3: CONN_01X03, Pin_Headers:Pin_Header_Angled_1x03, symbol CONN_01X03
- Y1: footprint Crystals:crystal_FA238-TSX3225 -> opendous:Crystal_5x3.2mm
Connections:
- net HTX0N is gone; now on net HTX0_N: P1.11 (P11)
- net HTX0P is gone; now on net HTX0_P: P1.9 (P9)
- net HTX1N is gone; now on net HTX1_N: P1.7 (P7)
- net HTX1P is gone; now on net HTX1_P: P1.5 (P5)
- net HTX2N is gone; now on net HTX2_N: P1.3 (P3)
- net HTX2P is gone; now on net HTX2_P: P1.1 (P1)
- net HTXCN is gone; now on net HTXC_N: P1.15 (P15)
- net HTXCP is gone; now on net HTXC_P: P1.13 (P13)
- net MICIN1 is gone; now on net UD0_P: P1.4 (P4)
- net GND: now also P3.1 (P1)
- net HCEC: now also U1.F21 (HCEC)
- net HHPD: now also U1.E21 (HHPD)
- net HSCL: now also U1.G21 (HSCL)
- net HSDA: now also U1.E20 (HSDA)
- net UD0_P: no longer P1.8 (P8)
- net UD1_N: now also U1.C22 (USB1-DM)
- net UD1_P: now also P1.8 (P8), U1.B23 (USB1-DP); no longer P1.12 (P12)
- net VCC_11: no longer P2.3 (P3), U1.AA1 (VDD-CPUX1), U1.AA3 (VDD-CPUX10), U1.AB2 (VDD-CPUX5), U1.AC1 (VDD-CPUX2), U1.AC2 (VDD-CPUX6), U1.H15 (VDD-CPUS), U1.J12 (VDD-SYS0), U1.J13 (VDD-SYS1), U1.K14 (VDD-SYS5), U1.K16 (HSIC-VCC), U1.L13 (VDD-SYS2), U1.L14 (VDD-SYS6), U1.M13 (VDD-SYS3), U1.M14 (VDD-SYS7), U1.N14 (VDD-SYS8), U1.P14 (VDD-SYS9), U1.R13 (VDD-SYS4), U1.R14 (VDD-SYS10), U1.T15 (VDD-SYS11), U1.U6 (VDD-CPUX16), U1.V2 (VDD-CPUX3), U1.V3 (VDD-CPUX7), U1.V4 (VDD-CPUX11), U1.V5 (VDD-CPUX14), U1.V6 (VDD-CPUX17), U1.W1 (VDD-CPUX0), U1.W3 (VDD-CPUX8), U1.W4 (VDD-CPUX12), U1.W5 (VDD-CPUX15), U1.Y2 (VDD-CPUX4), U1.Y3 (VDD-CPUX9), U1.Y4 (VDD-CPUX13)
- net VCC_15: now also P2.7 (P7); no longer P2.5 (P5)
- net VCC_30: no longer P2.7 (P7), U1.H16 (VCC-RTC), U1.N16 (VCC-PLL)
- net VCC_33: now also P2.5 (P5), U1.N16 (VCC-PLL); no longer P2.1 (P1)
- net HTX2_P: now reaches U1.D23 (HTX2P)
- net HTX2_N: now reaches U1.E22 (HTX2N)
- net HTX1_P: now reaches U1.E23 (HTX1P)
- net HTX1_N: now reaches U1.F22 (HTX1N)
- net HTX0_P: now reaches U1.G22 (HTX0P)
- net HTX0_N: now reaches U1.G23 (HTX0N)
- net HTXC_P: now reaches U1.H22 (HTXCP)
- net HTXC_N: now reaches U1.H23 (HTXCN)
- net UART1_TX: now reaches U1.AB17 (PG6/UART1-TX/PG_EINT6)
- net UART1_TX: now also P2.17 (P17)
- net UART1_RX: now reaches U1.U23 (PG7/UART1-RX/PG_EINT7)
- net UART1_RX: now also P2.15 (P15)
- net UART2_RX: now reaches U1.AB7 (PB1/UART2-RX/JTAG-CK0/PB_EINT1)
- net UART2_TX: now reaches U1.V9 (PB0/UART2-TX/JTAG-MS0/PB_EINT0)
- net HPCOM renamed VCC_13_RTC
- net VCC_13_RTC: now also U1.H16 (VCC-RTC)
- net HPL renamed VCC_30_ANL
- net HPR: no longer names the net of P2.13 (P13)
- net SATA_RXM: no longer names the net of P2.8 (P8)
- net SATA_RXP: no longer names the net of P2.6 (P6)
- net SATA_TXM: no longer names the net of P2.4 (P4)
- net SATA_TXP: no longer names the net of P2.2 (P2)
- net UART0_RX renamed UART3_RX
- net UART3_RX: now also P3.3 (P3); no longer P2.15 (P15)
- net UART0_TX renamed UART3_TX
- net UART3_TX: now also P3.2 (P2); no longer P2.17 (P17)
- net UD2_N: no longer names the net of P1.14 (P14)
- net UD2_N: no longer U1.C22 (USB1-DM)
- net UD2_P: no longer names the net of P1.16 (P16)
- net UD2_P: no longer U1.B23 (USB1-DP)
- new net VCC_11_CPU: P2.1 (P1), U1.AA1 (VDD-CPUX1), U1.AA3 (VDD-CPUX10), U1.AB2 (VDD-CPUX5), U1.AC1 (VDD-CPUX2), U1.AC2 (VDD-CPUX6), U1.H15 (VDD-CPUS), U1.U6 (VDD-CPUX16), U1.V2 (VDD-CPUX3), U1.V3 (VDD-CPUX7), U1.V4 (VDD-CPUX11), U1.V5 (VDD-CPUX14), U1.V6 (VDD-CPUX17), U1.W1 (VDD-CPUX0), U1.W3 (VDD-CPUX8), U1.W4 (VDD-CPUX12), U1.W5 (VDD-CPUX15), U1.Y2 (VDD-CPUX4), U1.Y3 (VDD-CPUX9), U1.Y4 (VDD-CPUX13)
- new net VCC_11_INT: P2.3 (P3), U1.J12 (VDD-SYS0), U1.J13 (VDD-SYS1), U1.K14 (VDD-SYS5), U1.K16 (HSIC-VCC), U1.L13 (VDD-SYS2), U1.L14 (VDD-SYS6), U1.M13 (VDD-SYS3), U1.M14 (VDD-SYS7), U1.N14 (VDD-SYS8), U1.P14 (VDD-SYS9), U1.R13 (VDD-SYS4), U1.R14 (VDD-SYS10), U1.T15 (VDD-SYS11)
Changed lines of the file:
@@
 	19500 8100 19500 8350
 Wire Wire Line
-	19500 8700 19500 8550
+	19500 8550 19500 8700
 Wire Wire Line
 	20300 8100 20300 8350
@@
 Connection ~ 19500 8300
 Wire Wire Line
-	19350 8350 19350 8300
+	19350 8300 19350 8350
 Connection ~ 19350 8300
 Wire Wire Line
@@
 Connection ~ 19500 8600
 Wire Wire Line
-	19350 8550 19350 8600
+	19350 8600 19350 8550
 Connection ~ 19350 8600
 Wire Wire Line
@@
 $EndComp
 Text GLabel 19100 9600 0    60   Input ~ 0
-HTX2P
+HTX2_P
 Text GLabel 19100 9700 0    60   Input ~ 0
-HTX2N
+HTX2_N
 Text GLabel 19100 9800 0    60   Input ~ 0
-HTX1P
+HTX1_P
 Text GLabel 19100 9900 0    60   Input ~ 0
-HTX1N
+HTX1_N
 Text GLabel 19100 10000 0    60   Input ~ 0
-HTX0P
+HTX0_P
 Text GLabel 19100 10100 0    60   Input ~ 0
-HTX0N
+HTX0_N
 Text GLabel 19100 10200 0    60   Input ~ 0
-HTXCP
+HTXC_P
 Text GLabel 19100 10300 0    60   Input ~ 0
-HTXCN
+HTXC_N
 Text GLabel 19100 10400 0    60   Input ~ 0
 HCEC
 Text GLabel 19100 10500 0    60   Input ~ 0
 HSCL
-Text GLabel 19600 9700 2    60   Input ~ 0
-MICIN1
 Text GLabel 19600 9800 2    60   Input ~ 0
 UD0_N
-Text GLabel 19600 9900 2    60   Input ~ 0
+Text GLabel 19600 9700 2    60   Input ~ 0
 UD0_P
 Text GLabel 19600 10000 2    60   Input ~ 0
 UD1_N
-Text GLabel 19600 10100 2    60   Input ~ 0
+Text GLabel 19600 9900 2    60   Input ~ 0
 UD1_P
-Text GLabel 19600 10200 2    60   Input ~ 0
-UD2_N
-Text GLabel 19600 10300 2    60   Input ~ 0
-UD2_P
 Text GLabel 19600 10400 2    60   Input ~ 0
 HHPD
@@
 	19600 9450 19800 9450
 Text GLabel 20650 9600 0    60   Input ~ 0
-VCC_33
+VCC_11_CPU
 Text GLabel 20650 9700 0    60   Input ~ 0
-VCC_11
+VCC_11_INT
 Text GLabel 20650 9800 0    60   Input ~ 0
+VCC_33
+Text GLabel 20650 9900 0    60   Input ~ 0
 VCC_15
-Text GLabel 20650 9900 0    60   Input ~ 0
-VCC_30
-Text GLabel 20650 10000 0    60   Input ~ 0
-HPCOM
-Text GLabel 20650 10100 0    60   Input ~ 0
-HPL
-Text GLabel 20650 10200 0    60   Input ~ 0
-HPR
 Text GLabel 20650 10300 0    60   Input ~ 0
-UART0_RX
+UART1_RX
 Text GLabel 20650 10400 0    60   Input ~ 0
-UART0_TX
+UART1_TX
 $Comp
 L GND #PWR09
@@
 Text GLabel 21150 10500 2    60   Input ~ 0
 SDC0_D2
-Text GLabel 21150 9600 2    60   Input ~ 0
-SATA_TXP
-Text GLabel 21150 9700 2    60   Input ~ 0
-SATA_TXM
-Text GLabel 21150 9800 2    60   Input ~ 0
-SATA_RXP
-Text GLabel 21150 9900 2    60   Input ~ 0
-SATA_RXM
 Text GLabel 17050 2750 2    60   Input ~ 0
 SA14
@@
 UD0_P
 Text GLabel 6350 8100 2    60   Input ~ 0
-UD2_N
+UD1_N
 Text GLabel 6350 8200 2    60   Input ~ 0
-UD2_P
+UD1_P
 Wire Wire Line
 	1650 2050 1650 2100
@@
 F 0 "Y1" H 1200 2200 50  0000 C CNN
 F 1 "Crystal" H 1200 1900 50  0000 C CNN
-F 2 "Crystals:crystal_FA238-TSX3225" H 1200 2050 50  0000 C CNN
+F 2 "opendous:Crystal_5x3.2mm" H 1200 2050 50  0000 C CNN
 F 3 "" H 1200 2050 50  0000 C CNN
 	1    1200 2050
@@
 $EndComp
 Text GLabel 6350 8800 2    60   Input ~ 0
-UART0_TX
+UART3_TX
 Text GLabel 6350 8900 2    60   Input ~ 0
-UART0_RX
+UART3_RX
 $Comp
 L GND #PWR012
@@
 $EndComp
 Wire Wire Line
-	8250 15850 8250 9750
+	8250 9750 8250 15850
 Wire Wire Line
 	8250 9750 8400 9750
@@
 Connection ~ 8250 15750
 Wire Wire Line
-	9800 12350 9900 12350
-Wire Wire Line
-	9900 12350 9900 10650
+	9900 12350 9800 12350
+Wire Wire Line
+	9900 10650 9900 12350
 Wire Wire Line
 	9900 10650 9800 10650
 Text GLabel 9900 10650 2    60   Input ~ 0
-VCC_11
+VCC_11_CPU
 Wire Wire Line
 	9800 10750 9900 10750
@@
 Connection ~ 9950 15650
 Wire Wire Line
-	10050 5950 9950 5950
-Wire Wire Line
-	9950 5950 9950 4950
+	9950 5950 10050 5950
+Wire Wire Line
+	9950 4950 9950 5950
 Wire Wire Line
 	9950 4950 10050 4950
@@
 Connection ~ 9900 14150
 Text GLabel 9900 13150 2    60   Input ~ 0
-VCC_11
+VCC_11_INT
 Text GLabel 6350 7800 2    60   Input ~ 0
 VCC_33
@@
 VCC_33
 Text GLabel 3050 1700 2    60   Input ~ 0
-VCC_11
+VCC_11_INT
 Text GLabel 3050 2100 2    60   Input ~ 0
 VCC_33
 Text GLabel 3050 2400 2    60   Input ~ 0
-VCC_30
+VCC_13_RTC
 Text GLabel 3050 2700 2    60   Input ~ 0
-VCC_30
+VCC_33
 Text GLabel 1500 7950 0    60   Input ~ 0
 VCC_30
 Text GLabel 9800 10250 2    60   Input ~ 0
-VCC_11
+VCC_11_CPU
 Wire Wire Line
 	9800 9750 9900 9750
@@
 Text GLabel 9900 9750 2    60   Input ~ 0
 VCC_33
+Text GLabel 20650 10000 0    60   Input ~ 0
+VCC_13_RTC
+Text GLabel 20650 10100 0    60   Input ~ 0
+VCC_30_ANL
+Text GLabel 4550 7800 0    60   Input ~ 0
+HTXC_P
+Text GLabel 4550 7900 0    60   Input ~ 0
+HTXC_N
+Text GLabel 4550 8000 0    60   Input ~ 0
+HTX0_P
+Text GLabel 4550 8100 0    60   Input ~ 0
+HTX0_N
+Text GLabel 4550 8200 0    60   Input ~ 0
+HTX1_P
+Text GLabel 4550 8300 0    60   Input ~ 0
+HTX1_N
+Text GLabel 4550 8400 0    60   Input ~ 0
+HTX2_P
+Text GLabel 4550 8500 0    60   Input ~ 0
+HTX2_N
+Text GLabel 4550 8600 0    60   Input ~ 0
+HCEC
+Text GLabel 4550 8700 0    60   Input ~ 0
+HHPD
+Text GLabel 4550 8800 0    60   Input ~ 0
+HSCL
+Text GLabel 4550 8900 0    60   Input ~ 0
+HSDA
+$Comp
+L CONN_01X03 P3
+U 1 1 56B45F5B
+P 17350 9750
+F 0 "P3" H 17350 9950 50  0000 C CNN
+F 1 "CONN_01X03" V 17450 9750 50  0000 C CNN
+F 2 "Pin_Headers:Pin_Header_Angled_1x03" H 17350 9750 50  0000 C CNN
+F 3 "" H 17350 9750 50  0000 C CNN
+	1    17350 9750
+	-1   0    0    1
+$EndComp
+Text GLabel 17550 9650 2    60   Input ~ 0
+UART3_RX
+Text GLabel 17550 9750 2    60   Input ~ 0
+UART3_TX
+$Comp
+L GND #PWR014
+U 1 1 56B46376
+P 17650 9900
+F 0 "#PWR014" H 17650 9650 50  0001 C CNN
+F 1 "GND" H 17650 9750 50  0000 C CNN
+F 2 "" H 17650 9900 50  0000 C CNN
+F 3 "" H 17650 9900 50  0000 C CNN
+	1    17650 9900
+	1    0    0    -1
+$EndComp
+Wire Wire Line
+	17550 9850 17650 9850
+Wire Wire Line
+	17650 9850 17650 9900
+Text GLabel 7150 11950 2    60   Input ~ 0
+UART2_TX
+Text GLabel 7150 12050 2    60   Input ~ 0
+UART2_RX
+Text GLabel 10750 7750 2    60   Input ~ 0
+UART1_TX
+Text GLabel 10750 7850 2    60   Input ~ 0
+UART1_RX
 $EndSCHEMATC
