File: tinycom-hdmi/tinycom-hdmi.kicad_pcb (KiCad board)
At the start: 2 copper layers, 45.2 x 45.2 mm, 47 parts, among them J1 MICRO_SD_HINGE, P1 CONN_02X10, P2 CONN_02X10, P4 USB_OTG, U1 SY8008BAAC, U2 AXP209, U3 SY8008BAAC, U4 RTL8188, U5 rainsun-antenna

Commit message: before replace
Parts:
- added C11: NC, Capacitors_SMD:C_0402, F.Cu at (154.1, 113.0)
- added C18: 10pF, Capacitors_SMD:C_0402, F.Cu at (155.8, 112.5)
- added C19: NC, Capacitors_SMD:C_0402, F.Cu at (157.6, 113.3)
- added R11: 2K, Resistors_SMD:R_0805, B.Cu at (163.4, 98.6)
- added R12: 47K, Resistors_SMD:R_0805, B.Cu at (163.4, 96.5)
- added R5: 2K, Resistors_SMD:R_0805, B.Cu at (163.4, 100.6)
- added U6: RCLAMP0524P, tinycom:SLP2510P8, F.Cu at (157.6, 105.2)
- added U7: RCLAMP0524P, tinycom:SLP2510P8, F.Cu at (157.6, 102.1)
- added U8: RCLAMP0524P, tinycom:SLP2510P8, F.Cu at (157.6, 99.0)
- U5: footprint tinycom:rainsun-antenna -> tinycom:AN9520
- moved C12 6.92 mm to (127.1, 108.2), turned to 180 degrees
- moved R2 4.37 mm to (154.1, 92.2)
- moved L1 4.33 mm to (150.2, 91.3)
- moved R1 4.33 mm to (154.1, 90.2)
- moved L3 4.23 mm to (158.1, 91.0)
- moved R4 4.11 mm to (161.9, 92.5)
- moved R3 4.11 mm to (161.9, 90.4)
- moved C5 4.00 mm to (158.1, 88.1)
- moved C14 3.70 mm to (141.9, 102.4)
- moved C13 3.13 mm to (140.1, 101.9)
- moved C17 2.98 mm to (137.5, 101.9)
- moved U2 2.95 mm to (139.6, 95.2)
- moved U1 2.93 mm to (150.2, 95.2)
- moved U3 2.78 mm to (157.8, 95.0)
- moved C2 2.28 mm to (150.2, 88.1)
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Connections:
- HDMI1 pad 1: HTX2_P -> Net-(HDMI1-Pad1)
- HDMI1 pad 10: HTXC_P -> Net-(HDMI1-Pad10)
- HDMI1 pad 11: GND -> Net-(HDMI1-Pad11)
- HDMI1 pad 12: HTXC_N -> GND
- HDMI1 pad 13: HCEC -> Net-(HDMI1-Pad13)
- HDMI1 pad 15: HCSL -> GND
- HDMI1 pad 16: HSDA -> Net-(HDMI1-Pad16)
- HDMI1 pad 17: GND -> Net-(HDMI1-Pad17)
- HDMI1 pad 18: +5V -> GND
- HDMI1 pad 19: HHPD -> Net-(HDMI1-Pad19)
- HDMI1 pad 2: GND -> +5V
- HDMI1 pad 3: HTX2_N -> GND
- HDMI1 pad 4: HTX1_P -> Net-(HDMI1-Pad4)
- HDMI1 pad 5: GND -> Net-(HDMI1-Pad5)
- HDMI1 pad 6: HTX1_N -> Net-(HDMI1-Pad6)
- HDMI1 pad 7: HTX0_P -> Net-(HDMI1-Pad7)
- HDMI1 pad 8: GND -> Net-(HDMI1-Pad8)
- HDMI1 pad 9: HTX0_N -> GND
- U4 pad 5: Net-(U4-Pad5) -> GND
- U4 pad 6: Net-(U4-Pad6) -> Net-(C11-Pad2)
- U5 pad 1: Net-(U4-Pad6) -> Net-(C18-Pad1)
- U5 pad 2: Net-(U4-Pad5) -> Net-(U5-Pad2)
Routing:
- net +5V: track 59.7 -> 0.00 mm
- net Net-(D1-Pad2): track 53.8 -> 0.00 mm, vias 2 -> 0
- net GND: track 52.4 -> 1.36 mm, vias 8 -> 1
- net VCC_33: track 44.2 -> 0.00 mm, vias 3 -> 0
- net IPSOUT: track 42.6 -> 0.00 mm, vias 5 -> 0
- net VCC_12_INT: track 38.8 -> 0.00 mm
- net HTX2_P: track 33.2 -> 0.00 mm, vias 1 -> 0
- net HTX2_N: track 32.4 -> 0.00 mm, vias 1 -> 0
- net HTX1_P: track 27.8 -> 0.00 mm, vias 1 -> 0
- net HTX1_N: track 27.3 -> 0.00 mm, vias 1 -> 0
- net UD0_N: track 27.1 -> 0.00 mm
- net UD0_P: track 26.5 -> 0.00 mm
- net SDC0_D1: track 25.9 -> 0.00 mm
- net VCC_12_CPU: track 25.8 -> 0.00 mm
- net SDC0_D0: track 25.4 -> 0.00 mm
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Other:
- net class Default: clearance 0.14 -> 0.15; trace_width 0.15 -> 0.4
- rule trace_clearance: 0.14 -> 0.15
