File: tinycom-hdmi/tinycom-hdmi.sch (KiCad schematic (older format))
At the start: 65 parts, among them J1 MICRO_SD_HINGE, P1 CONN_02X10, P2 CONN_02X10, P4 USB_OTG, U1 SY8008BAAC, U2 AXP209, U3 SY8008BAAC, U4 RTL8188, U5 rainsun-antenna, U6 RCLAMP0524P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

Commit message: hdmi route
Parts:
- added C27, C28: 10uF, Capacitors_SMD:C_1206, symbol C_Small
Connections:
- net GND: now also C27.2, C28.2
- net IPSOUT: now also C27.1, C28.1

Commit message: improve hdmi
Parts:
- added C29: 10uF, Capacitors_SMD:C_1206, symbol C_Small
- added C30, C31: C_Small, Capacitors_SMD:C_0805, symbol C_Small
- added L5, L6: SMD-FERRITE-BEAD-200R-2A(0805), OPL-Inductor-L0805, symbol SMD-FERRITE-BEAD-200R-2A(0805)
- R10: value 200K -> 2K
Connections:
- net UART1_RX is gone; now on net LDO4_28: P2.15 (P15)
- net +5V: now also HDMI1.18, C29.2; no longer HDMI1.2
- net GND: now also HDMI1.11, HDMI1.17, HDMI1.2, HDMI1.5, HDMI1.8, C29.1, C30.2, C31.2, L5.1, L6.2; no longer HDMI1.12, HDMI1.15, HDMI1.18, HDMI1.3, HDMI1.9, P4.6 (shield)
- net HCEC: now also U6.6 (OUT4); no longer U8.10 (OUT1)
- net HCSL: now also U6.7 (OUT3); no longer U8.9 (OUT2)
- net HHPD: now also U6.10 (OUT1); no longer U8.6 (OUT4)
- net HSDA: now also U6.9 (OUT2); no longer U8.7 (OUT3)
- net HTX0_N: now also U7.7 (OUT3); no longer U7.9 (OUT2)
- net HTX0_P: now also U7.6 (OUT4); no longer U7.10 (OUT1)
- net HTX1_N: now also U8.10 (OUT1); no longer U6.6 (OUT4)
- net HTX1_P: now also U8.9 (OUT2); no longer U6.7 (OUT3)
- net HTX2_N: now also U8.7 (OUT3); no longer U6.9 (OUT2)
- net HTX2_P: now also U8.6 (OUT4); no longer U6.10 (OUT1)
- net HTXC_N: now also U7.10 (OUT1); no longer U7.6 (OUT4)
- net HTXC_P: now also U7.9 (OUT2); no longer U7.7 (OUT3)
- net LDO3_28: now reaches P2.13 (P13)
- net LDO3_28: now also U2.41 (LDO3), C30.1
- net LDO4_28: now reaches U2.11 (LDO4)
- net LDO4_28: now also C31.1
- net at HDMI1.1, U8.5 (IN4): no longer R12.2
- net at HDMI1.10: now also U7.2 (IN2); no longer U7.4 (IN3)
- net at U7.1 (IN1): now also HDMI1.12; no longer HDMI1.13
- net at U6.5 (IN4): now also HDMI1.13; no longer HDMI1.14
- net at U6.4 (IN3): now also HDMI1.15, R11.1; no longer HDMI1.16
- net at U6.2 (IN2): now also HDMI1.16, R5.2; no longer HDMI1.17
- net at HDMI1.19, U6.1 (IN1): now also R12.2
- net at HDMI1.6: now also U8.1 (IN1)
- net at HDMI1.7: now also U7.5 (IN4); no longer U8.1 (IN1)
- net at HDMI1.SH1 (20): now also HDMI1.SH2 (21), HDMI1.SH3 (22), HDMI1.SH4 (23), L5.2
- net UART1_TX: no longer names the net of P2.17 (P17)
- new net: L6.1, P4.6 (shield)
- new net: HDMI1.3, U8.4 (IN3)
- new net: HDMI1.4, U8.2 (IN2)
- new net: HDMI1.9, U7.4 (IN3)
- no-connect marks 14 -> 13
Other:
- note added: "TODO: check hdmi shield pins / ground"
- moved on the sheet: HDMI1, R11, R12, R5, U6, U7, U8

Commit message: add mic to hdmi
Parts:
- added C32, C33: 10uF, Capacitors_SMD:C_0805, symbol C_Small
- added R20: 100K, Resistors_SMD:R_0805, symbol R_Small
- added U10, U9: admp411, tinycom:admp411, symbol admp411
Connections:
- net +3V3: now also C32.2, C33.2, U10.4 (LR), U10.7 (VDD), U10.8 (CHIPEN), U9.7 (VDD), U9.8 (CHIPEN)
- net GND: now also C32.1, C33.1, R20.1, U10.5 (GND), U10.6 (GND), U10.9 (GND), U9.4 (LR), U9.5 (GND), U9.6 (GND), U9.9 (GND)
- net I2S_SCK: now reaches P1.12 (P12)
- net I2S_SCK: now also U10.1 (SCK), U9.1 (SCK)
- net I2S_SD: now reaches P1.14 (P14)
- net I2S_SD: now also R20.2, U10.2 (SD), U9.2 (SD)
- net I2S_WS: now reaches P1.16 (P16)
- net I2S_WS: now also U10.3 (WS), U9.3 (WS)

Commit message: update hdmi
Parts:
- removed U6, U7, U8: RCLAMP0524P, tinycom:SLP2510P8, symbol RCLAMP0524P
Connections:
- net GND: now also C14.1
- net HCEC: now also HDMI1.13
- net HCSL: now also HDMI1.15, R11.1
- net HHPD: now also HDMI1.19, R12.2
- net HSDA: now also HDMI1.16, R5.2
- net HTX0_N: now also HDMI1.9
- net HTX0_P: now also HDMI1.7
- net HTX1_N: now also HDMI1.6
- net HTX1_P: now also HDMI1.4
- net HTX2_N: now also HDMI1.3
- net HTX2_P: now also HDMI1.1
- net HTXC_N: now also HDMI1.12
- net HTXC_P: now also HDMI1.10
