File: tinycom-audio/tinycom-audio.kicad_pcb (KiCad board)
At the start: 2 copper layers, 45.2 x 45.2 mm, 73 parts, among them J1 MICRO_SD_HINGE, P1 CONN_02X10, P2 CONN_02X10, P4 USB_OTG, U1 SY8008BAAC, U2 AXP209, U3 SY8008BAAC, U4 RTL8188, U5 rainsun-antenna, U6 admp411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

Commit message: update audio
Parts:
- removed R5: 100K, Resistors_SMD:R_0805
- added U8: audio-jack, tinycom:audio-jack, F.Cu at (165.1, 102.9)
- moved D1 46.1 mm to (126.4, 111.0)
- moved R9 44.6 mm to (129.5, 110.9), turned to 0 degrees
- moved C29 12.6 mm to (167.4, 92.5), turned to 180 degrees
- moved U6 12.5 mm to (167.2, 89.4)
- moved C32 5.36 mm to (131.3, 114.5)
- moved L6 1.17 mm to (132.0, 108.2)
- moved BT1 0.42 mm to (134.4, 111.9)
Routing:
- net Net-(D1-Pad2): track 60.6 -> 20.5 mm
- net VCC_33: track 72.9 -> 101.4 mm, vias 2 -> 3
- net I2S_SCK: track 58.4 -> 68.9 mm
- net I2S_WS: track 67.3 -> 76.9 mm
- net I2S_SD: track 64.1 -> 72.4 mm
- net GND: track 105.5 -> 101.6 mm, vias 31 -> 30
- net (no net): track 1.32 -> 0.00 mm
- net Net-(D1-Pad1): track 2.09 -> 1.15 mm
- net Net-(L6-Pad1): track 11.1 -> 10.4 mm
Other:
- net class Power: trace_width 0.2 -> 0.4

Commit message: pics
Parts:
- moved U8 2.26 mm to (163.4, 101.4), turned to 180 degrees
Routing:
- net I2S_WS: track 76.9 -> 76.4 mm
- net I2S_SD: track 72.4 -> 71.9 mm
Changed lines of the file:
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@@
 (kicad_pcb (version 4) (host pcbnew 4.0.0-2.201511301920+6191~38~ubuntu14.04.1-stable)
   (general
-    (links 208)
-    (no_connects 7)
+    (links 206)
+    (no_connects 5)
     (area 124.384999 79.172999 169.747001 124.535001)
     (thickness 1.6)
@@
   )
   (module tinycom:audio-jack (layer F.Cu)
-    (at 165.067 102.922)
-    (fp_text reference U8 (at -0.69 -8.66) (layer F.SilkS)
+    (at 163.417 101.372 180)
+    (fp_text reference U8 (at -0.69 -8.66 180) (layer F.SilkS)
       (effects (font (size 1 1) (thickness 0.15)))
     )
-    (fp_text value audio-jack (at -1.04 -10.27) (layer F.Fab)
+    (fp_text value audio-jack (at -1.04 -10.27 180) (layer F.Fab)
       (effects (font (size 1 1) (thickness 0.15)))
     )
@@
     (fp_line (start 4.24 -6.95) (end 4.24 5.36) (layer F.SilkS) (width 0.15))
     (fp_line (start -5.83 -6.95) (end 4.24 -6.95) (layer F.SilkS) (width 0.15))
-    (pad 5 thru_hole rect (at 2.94 4.32 180) (size 1.5 0.8) (drill 0.762) (layers *.Cu *.Mask F.SilkS)
+    (pad 5 thru_hole rect (at 2.94 4.32) (size 1.5 0.8) (drill 0.762) (layers *.Cu *.Mask F.SilkS)
       (net 73 "Net-(U8-Pad5)"))
-    (pad 2 thru_hole rect (at 2.94 -5.68 180) (size 1.5 0.8) (drill 0.762) (layers *.Cu *.Mask F.SilkS)
+    (pad 2 thru_hole rect (at 2.94 -5.68) (size 1.5 0.8) (drill 0.762) (layers *.Cu *.Mask F.SilkS)
       (net 74 "Net-(U8-Pad2)"))
-    (pad 3 thru_hole rect (at 2.94 -3.18 180) (size 1.5 0.8) (drill 0.762) (layers *.Cu *.Mask F.SilkS)
+    (pad 3 thru_hole rect (at 2.94 -3.18) (size 1.5 0.8) (drill 0.762) (layers *.Cu *.Mask F.SilkS)
       (net 75 "Net-(U8-Pad3)"))
-    (pad 4 thru_hole rect (at 2.94 1.82 180) (size 1.5 0.8) (drill 0.762) (layers *.Cu *.Mask F.SilkS)
+    (pad 4 thru_hole rect (at 2.94 1.82) (size 1.5 0.8) (drill 0.762) (layers *.Cu *.Mask F.SilkS)
       (net 76 "Net-(U8-Pad4)"))
-    (pad 1 thru_hole rect (at -2.06 -0.68 270) (size 1.5 0.8) (drill 0.762) (layers *.Cu *.Mask F.SilkS)
+    (pad 1 thru_hole rect (at -2.06 -0.68 90) (size 1.5 0.8) (drill 0.762) (layers *.Cu *.Mask F.SilkS)
       (net 77 "Net-(U8-Pad1)"))
-    (pad NC thru_hole circle (at -2.06 4.32 270) (size 1.2 1.2) (drill 1.2) (layers *.Cu *.Mask F.SilkS))
-    (pad NC thru_hole circle (at -2.1 -5.71 270) (size 1.2 1.2) (drill 1.2) (layers *.Cu *.Mask F.SilkS))
-    (pad NC thru_hole circle (at -4.56 -5.68 270) (size 1.2 1.2) (drill 1.2) (layers *.Cu *.Mask F.SilkS))
-    (pad NC thru_hole circle (at -4.56 4.32 270) (size 1.2 1.2) (drill 1.2) (layers *.Cu *.Mask F.SilkS))
+    (pad NC thru_hole circle (at -2.06 4.32 90) (size 1.2 1.2) (drill 1.2) (layers *.Cu *.Mask F.SilkS))
+    (pad NC thru_hole circle (at -2.1 -5.71 90) (size 1.2 1.2) (drill 1.2) (layers *.Cu *.Mask F.SilkS))
+    (pad NC thru_hole circle (at -4.56 -5.68 90) (size 1.2 1.2) (drill 1.2) (layers *.Cu *.Mask F.SilkS))
+    (pad NC thru_hole circle (at -4.56 4.32 90) (size 1.2 1.2) (drill 1.2) (layers *.Cu *.Mask F.SilkS))
   )
   (gr_text "rev. 1" (at 166.117 102.242 90) (layer B.SilkS)
@@
   (via (at 131.147 90.742) (size 0.6) (drill 0.3) (layers F.Cu B.Cu) (net 68))
   (via (at 135.75 87.25) (size 0.6) (drill 0.3) (layers F.Cu B.Cu) (net 68))
-  (segment (start 148.267 120.482) (end 147.163399 119.378399) (width 0.2) (layer F.Cu) (net 70))
-  (segment (start 147.163399 119.378399) (end 147.163399 109.246601) (width 0.2) (layer F.Cu) (net 70))
-  (segment (start 147.163399 109.246601) (end 155.748 100.662) (width 0.2) (layer F.Cu) (net 70))
-  (segment (start 155.748 100.662) (end 162.008 100.662) (width 0.2) (layer F.Cu) (net 70))
-  (segment (start 162.008 100.662) (end 163.807001 98.862999) (width 0.2) (layer F.Cu) (net 70))
-  (segment (start 163.807001 98.862999) (end 163.807001 90.291999) (width 0.2) (layer F.Cu) (net 70))
   (segment (start 165.457 88.642) (end 165.457 88.142) (width 0.2) (layer F.Cu) (net 70))
   (segment (start 163.807001 90.291999) (end 165.457 88.642) (width 0.2) (layer F.Cu) (net 70))
+  (segment (start 155.748 100.662) (end 161.166304 100.662) (width 0.2) (layer F.Cu) (net 70))
+  (segment (start 147.163399 119.378399) (end 147.163399 109.246601) (width 0.2) (layer F.Cu) (net 70))
+  (segment (start 147.163399 109.246601) (end 155.748 100.662) (width 0.2) (layer F.Cu) (net 70))
+  (segment (start 148.267 120.482) (end 147.163399 119.378399) (width 0.2) (layer F.Cu) (net 70))
+  (segment (start 163.807001 98.021303) (end 163.807001 90.291999) (width 0.2) (layer F.Cu) (net 70))
+  (segment (start 161.166304 100.662) (end 163.807001 98.021303) (width 0.2) (layer F.Cu) (net 70))
   (segment (start 128.717 115.372) (end 129.675 116.33) (width 0.2) (layer F.Cu) (net 70))
   (segment (start 147.403401 121.345599) (end 148.267 120.482) (width 0.2) (layer F.Cu) (net 70))
@@
   (segment (start 133.933412 121.973412) (end 146.775588 121.973412) (width 0.2) (layer F.Cu) (net 70))
   (segment (start 146.775588 121.973412) (end 147.403401 121.345599) (width 0.2) (layer F.Cu) (net 70))
-  (segment (start 164.557 90.762) (end 164.557 99.109998) (width 0.2) (layer F.Cu) (net 71))
-  (segment (start 164.557 99.109998) (end 161.546998 102.12) (width 0.2) (layer F.Cu) (net 71))
-  (segment (start 161.546998 102.12) (end 155.65 102.12) (width 0.2) (layer F.Cu) (net 71))
-  (segment (start 155.65 102.12) (end 150.78 106.99) (width 0.2) (layer F.Cu) (net 71))
   (segment (start 150.78 106.99) (end 150.78 116.16) (width 0.2) (layer F.Cu) (net 71))
   (segment (start 150.78 116.16) (end 152.13 117.51) (width 0.2) (layer F.Cu) (net 71))
+  (segment (start 156.28 101.49) (end 150.78 106.99) (width 0.2) (layer F.Cu) (net 71))
   (segment (start 152.13 117.51) (end 152.13 119.265) (width 0.2) (layer F.Cu) (net 71))
   (segment (start 152.13 119.265) (end 153.347 120.482) (width 0.2) (layer F.Cu) (net 71))
+  (segment (start 164.557 90.762) (end 164.557 98.233) (width 0.2) (layer F.Cu) (net 71))
+  (segment (start 164.557 98.233) (end 161.3 101.49) (width 0.2) (layer F.Cu) (net 71))
+  (segment (start 161.3 101.49) (end 156.28 101.49) (width 0.2) (layer F.Cu) (net 71))
   (segment (start 166.644997 88.682001) (end 167.116999 88.682001) (width 0.2) (layer F.Cu) (net 71))
   (segment (start 167.557 88.242) (end 167.557 88.142) (width 0.2) (layer F.Cu) (net 71))
@@
   (segment (start 151.175567 122.653433) (end 152.483401 121.345599) (width 0.2) (layer F.Cu) (net 71))
   (segment (start 152.483401 121.345599) (end 153.347 120.482) (width 0.2) (layer F.Cu) (net 71))
-  (segment (start 166.507 88.242) (end 166.507 88.142) (width 0.2) (layer F.Cu) (net 72))
-  (segment (start 164.147013 99.039137) (end 164.147013 90.601987) (width 0.2) (layer F.Cu) (net 72))
-  (segment (start 155.848001 101.251999) (end 161.934151 101.251999) (width 0.2) (layer F.Cu) (net 72))
+  (segment (start 161.159163 101.149989) (end 164.147013 98.162139) (width 0.2) (layer F.Cu) (net 72))
+  (segment (start 164.147013 98.162139) (end 164.147013 90.601987) (width 0.2) (layer F.Cu) (net 72))
+  (segment (start 149.370601 107.729399) (end 155.950011 101.149989) (width 0.2) (layer F.Cu) (net 72))
   (segment (start 164.147013 90.601987) (end 166.507 88.242) (width 0.2) (layer F.Cu) (net 72))
-  (segment (start 161.934151 101.251999) (end 164.147013 99.039137) (width 0.2) (layer F.Cu) (net 72))
-  (segment (start 149.370601 107.729399) (end 155.848001 101.251999) (width 0.2) (layer F.Cu) (net 72))
-  (segment (start 149.370601 119.045601) (end 149.370601 107.729399) (width 0.2) (layer F.Cu) (net 72))
+  (segment (start 155.950011 101.149989) (end 161.159163 101.149989) (width 0.2) (layer F.Cu) (net 72))
   (segment (start 150.807 120.482) (end 149.370601 119.045601) (width 0.2) (layer F.Cu) (net 72))
+  (segment (start 166.507 88.242) (end 166.507 88.142) (width 0.2) (layer F.Cu) (net 72))
+  (segment (start 149.370601 119.045601) (end 149.370601 107.729399) (width 0.2) (layer F.Cu) (net 72))
   (segment (start 149.943401 121.345599) (end 150.807 120.482) (width 0.2) (layer F.Cu) (net 72))
   (segment (start 148.975577 122.313423) (end 149.943401 121.345599) (width 0.2) (layer F.Cu) (net 72))
